File: Quanta_v1/Quanta_v1.kicad_pcb (KiCad board)
At the start: 2 copper layers, 0 parts

Commit message: start pcb
Parts:
- added 6.25u stabilizer: Stabilizer_Cherry_MX_6.25u, PCM_Mounting_Keyboard_Stabilizer:Stabilizer_Cherry_MX_6.25u, F.Cu at (179.2, 213.0)
- added C1: 10uF, Capacitor_SMD:C_0805_2012Metric_Pad1.18x1.45mm_HandSolder, B.Cu at (399.9, 72.1)
- added C2: 10uF, Capacitor_SMD:C_0805_2012Metric_Pad1.18x1.45mm_HandSolder, B.Cu at (399.9, 75.1)
- added C3: 100nF, Capacitor_SMD:C_0805_2012Metric_Pad1.18x1.45mm_HandSolder, B.Cu at (399.9, 78.1)
- added C4: 10uF, Capacitor_SMD:C_0805_2012Metric_Pad1.18x1.45mm_HandSolder, B.Cu at (399.9, 81.1)
- added C5: 100uF, Capacitor_SMD:C_1206_3216Metric_Pad1.33x1.80mm_HandSolder, B.Cu at (394.5, 72.2)
- added C6: 100uF, Capacitor_SMD:C_1206_3216Metric_Pad1.33x1.80mm_HandSolder, B.Cu at (394.5, 75.6)
- added C7: 100nF, Capacitor_SMD:C_0805_2012Metric_Pad1.18x1.45mm_HandSolder, B.Cu at (399.9, 84.1)
- added C8: 100uF, Capacitor_SMD:C_1206_3216Metric_Pad1.33x1.80mm_HandSolder, B.Cu at (394.5, 78.9)
- added C9: 100uF, Capacitor_SMD:C_1206_3216Metric_Pad1.33x1.80mm_HandSolder, B.Cu at (394.5, 82.3)
- added D1: DIODE, Diode_SMD:D_SOD-123, B.Cu at (64.0, 116.5)
- added D10: DIODE, Diode_SMD:D_SOD-123, B.Cu at (249.8, 116.5)
- added D11: DIODE, Diode_SMD:D_SOD-123, B.Cu at (268.8, 116.5)
- added D12: DIODE, Diode_SMD:D_SOD-123, B.Cu at (287.9, 116.5)
- added D13: DIODE, Diode_SMD:D_SOD-123, B.Cu at (306.9, 116.5)
- added D14: DIODE, Diode_SMD:D_SOD-123, B.Cu at (64.0, 140.3)
- added D15: DIODE, Diode_SMD:D_SOD-123, B.Cu at (83.1, 140.3)
- added D16: DIODE, Diode_SMD:D_SOD-123, B.Cu at (102.2, 140.3)
- added D17: DIODE, Diode_SMD:D_SOD-123, B.Cu at (121.2, 140.3)
- added D18: DIODE, Diode_SMD:D_SOD-123, B.Cu at (140.2, 140.3)
- added D19: DIODE, Diode_SMD:D_SOD-123, B.Cu at (159.3, 140.3)
- added D2: DIODE, Diode_SMD:D_SOD-123, B.Cu at (87.9, 116.5)
- added D20: DIODE, Diode_SMD:D_SOD-123, B.Cu at (178.3, 140.3)
- added D21: DIODE, Diode_SMD:D_SOD-123, B.Cu at (197.4, 140.3)
- added D22: DIODE, Diode_SMD:D_SOD-123, B.Cu at (216.4, 140.3)
- added D23: DIODE, Diode_SMD:D_SOD-123, B.Cu at (235.5, 140.3)
- added D24: DIODE, Diode_SMD:D_SOD-123, B.Cu at (254.6, 140.3)
- added D25: DIODE, Diode_SMD:D_SOD-123, B.Cu at (273.6, 140.3)
- added D26: DIODE, Diode_SMD:D_SOD-123, B.Cu at (292.6, 140.3)
- added D27: DIODE, Diode_SMD:D_SOD-123, B.Cu at (321.2, 140.3)
- added D28: DIODE, Diode_SMD:D_SOD-123, B.Cu at (359.3, 140.3)
- added D29: DIODE, Diode_SMD:D_SOD-123, B.Cu at (68.8, 159.4)
- added D3: DIODE, Diode_SMD:D_SOD-123, B.Cu at (106.9, 116.5)
- added D30: DIODE, Diode_SMD:D_SOD-123, B.Cu at (92.6, 159.4)
- added D31: DIODE, Diode_SMD:D_SOD-123, B.Cu at (111.7, 159.4)
- added D32: DIODE, Diode_SMD:D_SOD-123, B.Cu at (130.7, 159.4)
- added D33: DIODE, Diode_SMD:D_SOD-123, B.Cu at (149.8, 159.4)
- added D34: DIODE, Diode_SMD:D_SOD-123, B.Cu at (168.8, 159.4)
- added D35: DIODE, Diode_SMD:D_SOD-123, B.Cu at (187.9, 159.4)
- added D36: DIODE, Diode_SMD:D_SOD-123, B.Cu at (206.9, 159.4)
- added D37: DIODE, Diode_SMD:D_SOD-123, B.Cu at (226.0, 159.4)
- added D38: DIODE, Diode_SMD:D_SOD-123, B.Cu at (245.0, 159.4)
- added D39: DIODE, Diode_SMD:D_SOD-123, B.Cu at (264.1, 159.4)
- added D4: DIODE, Diode_SMD:D_SOD-123, B.Cu at (126.0, 116.5)
- added D40: DIODE, Diode_SMD:D_SOD-123, B.Cu at (283.1, 159.4)
- added D41: DIODE, Diode_SMD:D_SOD-123, B.Cu at (302.2, 159.4)
- added D42: DIODE, Diode_SMD:D_SOD-123, B.Cu at (328.4, 168.9)
- added D43: DIODE, Diode_SMD:D_SOD-123, B.Cu at (359.3, 159.4)
- added D44: DIODE, Diode_SMD:D_SOD-123, B.Cu at (71.2, 178.4)
- added D45: DIODE, Diode_SMD:D_SOD-123, B.Cu at (97.4, 178.4)
- added D46: DIODE, Diode_SMD:D_SOD-123, B.Cu at (116.4, 178.4)
- added D47: DIODE, Diode_SMD:D_SOD-123, B.Cu at (135.5, 178.4)
- added D48: DIODE, Diode_SMD:D_SOD-123, B.Cu at (154.5, 178.4)
- added D49: DIODE, Diode_SMD:D_SOD-123, B.Cu at (173.6, 178.4)
- added D5: DIODE, Diode_SMD:D_SOD-123, B.Cu at (145.0, 116.5)
- added D50: DIODE, Diode_SMD:D_SOD-123, B.Cu at (192.6, 178.4)
- added D51: DIODE, Diode_SMD:D_SOD-123, B.Cu at (211.7, 178.4)
- added D52: DIODE, Diode_SMD:D_SOD-123, B.Cu at (230.7, 178.4)
- added D53: DIODE, Diode_SMD:D_SOD-123, B.Cu at (249.8, 178.4)
- added D54: DIODE, Diode_SMD:D_SOD-123, B.Cu at (268.8, 178.4)
- added D55: DIODE, Diode_SMD:D_SOD-123, B.Cu at (287.9, 178.4)
- added D56: DIODE, Diode_SMD:D_SOD-123, B.Cu at (306.9, 178.4)
- added D57: DIODE, Diode_SMD:D_SOD-123, B.Cu at (359.3, 178.4)
- added D58: DIODE, Diode_SMD:D_SOD-123, B.Cu at (66.4, 197.5)
- added D59: DIODE, Diode_SMD:D_SOD-123, B.Cu at (87.9, 197.5)
- added D6: DIODE, Diode_SMD:D_SOD-123, B.Cu at (168.8, 116.5)
- added D60: DIODE, Diode_SMD:D_SOD-123, B.Cu at (106.9, 197.5)
- added D61: DIODE, Diode_SMD:D_SOD-123, B.Cu at (126.0, 197.5)
- added D62: DIODE, Diode_SMD:D_SOD-123, B.Cu at (145.0, 197.5)
- added D63: DIODE, Diode_SMD:D_SOD-123, B.Cu at (164.1, 197.5)
- added D64: DIODE, Diode_SMD:D_SOD-123, B.Cu at (183.1, 197.5)
- added D65: DIODE, Diode_SMD:D_SOD-123, B.Cu at (202.2, 197.5)
- added D66: DIODE, Diode_SMD:D_SOD-123, B.Cu at (221.2, 197.5)
- added D67: DIODE, Diode_SMD:D_SOD-123, B.Cu at (240.3, 197.5)
- added D68: DIODE, Diode_SMD:D_SOD-123, B.Cu at (259.3, 197.5)
- added D69: DIODE, Diode_SMD:D_SOD-123, B.Cu at (278.4, 197.5)
- added D7: DIODE, Diode_SMD:D_SOD-123, B.Cu at (187.9, 116.5)
- added D70: DIODE, Diode_SMD:D_SOD-123, B.Cu at (304.6, 197.5)
- added D71: DIODE, Diode_SMD:D_SOD-123, B.Cu at (359.3, 197.5)
- added D72: DIODE, Diode_SMD:D_SOD-123, B.Cu at (335.5, 202.2)
- added D73: DIODE, Diode_SMD:D_SOD-123, B.Cu at (66.4, 216.5)
- added D74: DIODE, Diode_SMD:D_SOD-123, B.Cu at (90.2, 216.5)
- added D75: DIODE, Diode_SMD:D_SOD-123, B.Cu at (114.1, 216.5)
- added D76: DIODE, Diode_SMD:D_SOD-123, B.Cu at (183.0, 221.6)
- added D77: DIODE, Diode_SMD:D_SOD-123, B.Cu at (254.6, 216.5)
- added D78: DIODE, Diode_SMD:D_SOD-123, B.Cu at (273.6, 216.5)
- added D79: DIODE, Diode_SMD:D_SOD-123, B.Cu at (292.6, 216.5)
- added D8: DIODE, Diode_SMD:D_SOD-123, B.Cu at (206.9, 116.5)
- added D80: DIODE, Diode_SMD:D_SOD-123, B.Cu at (316.5, 221.3)
- added D81: DIODE, Diode_SMD:D_SOD-123, B.Cu at (335.5, 221.3)
- added D82: DIODE, Diode_SMD:D_SOD-123, B.Cu at (354.6, 221.3)
- added D83: USBLC6-2SC6, Package_TO_SOT_SMD:SOT-23-6_Handsoldering, B.Cu at (324.5, 83.6)
- added D84: USBLC6-2SC6, Package_TO_SOT_SMD:SOT-23-6_Handsoldering, B.Cu at (326.1, 105.0)
- added D85: USBLC6-2SC6, Package_TO_SOT_SMD:SOT-23-6_Handsoldering, B.Cu at (359.0, 84.4)
- added D86: USBLC6-2SC6, Package_TO_SOT_SMD:SOT-23-6_Handsoldering, B.Cu at (340.7, 86.8)
- added D9: DIODE, Diode_SMD:D_SOD-123, B.Cu at (226.0, 116.5)
- added F1: 2A, Fuse:Fuse_1206_3216Metric_Pad1.42x1.75mm_HandSolder, B.Cu at (389.6, 24.6)
- added F2: 500mA, Fuse:Fuse_1206_3216Metric_Pad1.42x1.75mm_HandSolder, B.Cu at (389.6, 27.9)
- added F3: 500mA, Fuse:Fuse_1206_3216Metric_Pad1.42x1.75mm_HandSolder, B.Cu at (389.6, 31.2)
- added F4: 500mA, Fuse:Fuse_1206_3216Metric_Pad1.42x1.75mm_HandSolder, B.Cu at (389.6, 34.5)
- added FB1: 600R, PCM_Ferrite_SMD_Handsoldering_AKL:Ferrite_0805_2012Metric, B.Cu at (352.3, 72.6)
- added FB2: 600R, PCM_Ferrite_SMD_Handsoldering_AKL:Ferrite_0805_2012Metric, B.Cu at (221.0, 26.2)
- added FB3: 600R, PCM_Ferrite_SMD_Handsoldering_AKL:Ferrite_0805_2012Metric, B.Cu at (221.0, 29.3)
- added FB4: 100R 2A5, PCM_Ferrite_SMD_Handsoldering_AKL:Ferrite_0603_1608Metric, B.Cu at (274.0, 70.2)
- added FB5: 600R 500mA, PCM_Ferrite_SMD_Handsoldering_AKL:Ferrite_0805_2012Metric, B.Cu at (221.0, 32.4)
- added FB6: 600R 500mA, PCM_Ferrite_SMD_Handsoldering_AKL:Ferrite_0805_2012Metric, B.Cu at (221.0, 35.5)
- added FB7: 600R, PCM_Ferrite_SMD_Handsoldering_AKL:Ferrite_0805_2012Metric, B.Cu at (221.0, 38.6)
- added FB8: 600R 500mA, PCM_Ferrite_SMD_Handsoldering_AKL:Ferrite_0805_2012Metric, B.Cu at (221.0, 41.8)
- added J1: USB_C_Receptacle_USB2.0, USB_C_socket_GT-USB-7010H:USB-C-SMD_G-SWITCH_GT-USB-7010EN, B.Cu at (325.4, 65.1)
- added J10: USB_A_Receptacle_UBS2.0, USB_A_horizontal_SMD_903-231A2031S10100:USB-A-SMD_903-231A2031S10100, B.Cu at (342.9, 71.9)
- added J11: Conn_01x01_Socket GND, Connector_PinHeader_2.54mm:PinHeader_1x01_P2.54mm_Vertical, B.Cu at (273.8, 61.9)
- added J12: Conn_01x06_Socket GPIOs, Connector_PinHeader_2.54mm:PinHeader_1x06_P2.54mm_Vertical, B.Cu at (189.2, 67.5)
- added J13: Conn_01x01_Socket GPIO0, Connector_PinHeader_2.54mm:PinHeader_1x01_P2.54mm_Vertical, B.Cu at (273.8, 66.5)
- added J2: Conn_01x02_Socket VBUS 5V, Connector_PinHeader_2.54mm:PinHeader_1x02_P2.54mm_Vertical, B.Cu at (211.0, 77.8)
- added J3: Conn_01x02_Socket 3V3, Connector_PinHeader_2.54mm:PinHeader_1x02_P2.54mm_Vertical, B.Cu at (211.0, 83.3)
- added J4: Conn_01x02_Socket VBAT, Connector_PinHeader_2.54mm:PinHeader_1x02_P2.54mm_Vertical, B.Cu at (211.0, 72.2)
- added J5: Conn_01x04_Socket SWL, Connector_PinHeader_2.54mm:PinHeader_1x04_P2.54mm_Vertical, B.Cu at (273.8, 27.8)
- added J6: USB_A_Receptacle_UBS2.0, USB_A_vertical_KH-AF180ZJ-13.7:USB-A-TH_KH-AF180ZJ-13.7, F.Cu at (326.2, 112.7)
- added J7: JSTConn USB3, Connector_JST:JST_EH_S4B-EH_1x04_P2.50mm_Horizontal, B.Cu at (141.1, 71.6)
- added J8: JSTConn USB4, Connector_JST:JST_EH_S4B-EH_1x04_P2.50mm_Horizontal, B.Cu at (141.1, 82.0)
- added J9: USB_C_Receptacle_USB2.0, USB_C_socket_GT-USB-7010H:USB-C-SMD_G-SWITCH_GT-USB-7010EN, B.Cu at (360.4, 65.1)
- added JP1: SolderJumper-Bridged, Jumper:SolderJumper-2_P1.3mm_Bridged_RoundedPad1.0x1.5mm, B.Cu at (210.6, 49.6)
- added R1: 0R, Resistor_SMD:R_1206_3216Metric_Pad1.30x1.75mm_HandSolder, B.Cu at (389.6, 37.8)
- added R10: 56K 20%, Resistor_SMD:R_0603_1608Metric_Pad0.98x0.95mm_HandSolder, B.Cu at (274.0, 55.8)
- added R11: 56K 20%, Resistor_SMD:R_0603_1608Metric_Pad0.98x0.95mm_HandSolder, B.Cu at (274.0, 58.3)
- added R12: 0R, Resistor_SMD:R_1206_3216Metric_Pad1.30x1.75mm_HandSolder, B.Cu at (353.7, 70.1)
- added R13: 1M, Resistor_SMD:R_0805_2012Metric_Pad1.20x1.40mm_HandSolder, B.Cu at (352.4, 67.5)
- added R2: 0R, Resistor_SMD:R_1206_3216Metric_Pad1.30x1.75mm_HandSolder, B.Cu at (389.6, 41.1)
- added R3: 5K11, Resistor_SMD:R_0603_1608Metric_Pad0.98x0.95mm_HandSolder, B.Cu at (327.1, 70.4)
- added R4: 5K11, Resistor_SMD:R_0603_1608Metric_Pad0.98x0.95mm_HandSolder, B.Cu at (324.3, 70.4)
- added R5: 1M, Resistor_SMD:R_0805_2012Metric_Pad1.20x1.40mm_HandSolder, B.Cu at (273.8, 39.2)
- added R6: 1M, Resistor_SMD:R_0805_2012Metric_Pad1.20x1.40mm_HandSolder, B.Cu at (273.8, 42.1)
- added R8: 0R, Resistor_SMD:R_1206_3216Metric_Pad1.30x1.75mm_HandSolder, B.Cu at (389.6, 44.3)
- added R9: 1M, Resistor_SMD:R_0805_2012Metric_Pad1.20x1.40mm_HandSolder, B.Cu at (273.8, 45.1)
- added RED1: DIODE, Diode_SMD:D_SOD-123, B.Cu at (359.3, 124.6)
- added RESW1: RotaryEncoder_Switch, Rotary_Encoder:RotaryEncoder_Bourns_Vertical_PEC12R-3xxxF-Sxxxx, F.Cu at (355.4, 105.5)
- added SW1: SW_Push, Button_Switch_Keyboard:SW_Cherry_MX_1.00u_PCB, F.Cu at (60.3, 108.0)
- added SW10: SW_Push, Button_Switch_Keyboard:SW_Cherry_MX_1.00u_PCB, F.Cu at (246.1, 108.0)
- added SW11: SW_Push, Button_Switch_Keyboard:SW_Cherry_MX_1.00u_PCB, F.Cu at (265.1, 108.0)
- added SW12: SW_Push, Button_Switch_Keyboard:SW_Cherry_MX_1.00u_PCB, F.Cu at (284.2, 108.0)
- added SW13: SW_Push, Button_Switch_Keyboard:SW_Cherry_MX_1.00u_PCB, F.Cu at (303.2, 108.0)
- added SW14: SW_Push, Button_Switch_Keyboard:SW_Cherry_MX_1.00u_PCB, F.Cu at (60.3, 131.8)
- added SW15: SW_Push, Button_Switch_Keyboard:SW_Cherry_MX_1.00u_PCB, F.Cu at (79.4, 131.8)
- added SW16: SW_Push, Button_Switch_Keyboard:SW_Cherry_MX_1.00u_PCB, F.Cu at (98.4, 131.8)
- added SW17: SW_Push, Button_Switch_Keyboard:SW_Cherry_MX_1.00u_PCB, F.Cu at (117.5, 131.8)
- added SW18: SW_Push, Button_Switch_Keyboard:SW_Cherry_MX_1.00u_PCB, F.Cu at (136.5, 131.8)
- added SW19: SW_Push, Button_Switch_Keyboard:SW_Cherry_MX_1.00u_PCB, F.Cu at (155.6, 131.8)
- added SW2: SW_Push, Button_Switch_Keyboard:SW_Cherry_MX_1.00u_PCB, F.Cu at (84.1, 108.0)
- added SW20: SW_Push, Button_Switch_Keyboard:SW_Cherry_MX_1.00u_PCB, F.Cu at (174.6, 131.8)
- added SW21: SW_Push, Button_Switch_Keyboard:SW_Cherry_MX_1.00u_PCB, F.Cu at (193.7, 131.8)
- added SW22: SW_Push, Button_Switch_Keyboard:SW_Cherry_MX_1.00u_PCB, F.Cu at (212.7, 131.8)
- added SW23: SW_Push, Button_Switch_Keyboard:SW_Cherry_MX_1.00u_PCB, F.Cu at (231.8, 131.8)
- added SW24: SW_Push, Button_Switch_Keyboard:SW_Cherry_MX_1.00u_PCB, F.Cu at (250.8, 131.8)
- added SW25: SW_Push, Button_Switch_Keyboard:SW_Cherry_MX_1.00u_PCB, F.Cu at (269.9, 131.8)
- added SW26: SW_Push, Button_Switch_Keyboard:SW_Cherry_MX_1.00u_PCB, F.Cu at (288.9, 131.8)
- added SW27: SW_Push, Button_Switch_Keyboard:SW_Cherry_MX_2.00u_PCB, F.Cu at (317.5, 131.8)
- added SW28: SW_Push, Button_Switch_Keyboard:SW_Cherry_MX_1.00u_PCB, F.Cu at (355.6, 131.8)
- added SW29: SW_Push, Button_Switch_Keyboard:SW_Cherry_MX_1.50u_PCB, F.Cu at (65.1, 150.8)
- added SW3: SW_Push, Button_Switch_Keyboard:SW_Cherry_MX_1.00u_PCB, F.Cu at (103.2, 108.0)
- added SW30: SW_Push, Button_Switch_Keyboard:SW_Cherry_MX_1.00u_PCB, F.Cu at (88.9, 150.8)
- added SW31: SW_Push, Button_Switch_Keyboard:SW_Cherry_MX_1.00u_PCB, F.Cu at (108.0, 150.8)
- added SW32: SW_Push, Button_Switch_Keyboard:SW_Cherry_MX_1.00u_PCB, F.Cu at (127.0, 150.8)
- added SW33: SW_Push, Button_Switch_Keyboard:SW_Cherry_MX_1.00u_PCB, F.Cu at (146.1, 150.8)
- added SW34: SW_Push, Button_Switch_Keyboard:SW_Cherry_MX_1.00u_PCB, F.Cu at (165.1, 150.8)
- added SW35: SW_Push, Button_Switch_Keyboard:SW_Cherry_MX_1.00u_PCB, F.Cu at (184.2, 150.8)
- added SW36: SW_Push, Button_Switch_Keyboard:SW_Cherry_MX_1.00u_PCB, F.Cu at (203.2, 150.8)
- added SW37: SW_Push, Button_Switch_Keyboard:SW_Cherry_MX_1.00u_PCB, F.Cu at (222.2, 150.8)
- added SW38: SW_Push, Button_Switch_Keyboard:SW_Cherry_MX_1.00u_PCB, F.Cu at (241.3, 150.8)
- added SW39: SW_Push, Button_Switch_Keyboard:SW_Cherry_MX_1.00u_PCB, F.Cu at (260.4, 150.8)
- added SW4: SW_Push, Button_Switch_Keyboard:SW_Cherry_MX_1.00u_PCB, F.Cu at (122.2, 108.0)
- added SW40: SW_Push, Button_Switch_Keyboard:SW_Cherry_MX_1.00u_PCB, F.Cu at (279.4, 150.8)
- added SW41: SW_Push, Button_Switch_Keyboard:SW_Cherry_MX_1.00u_PCB, F.Cu at (298.4, 150.8)
- added SW42: SW_Push, Button_Switch_Keyboard:SW_Cherry_MX_ISOEnter_PCB, F.Cu at (324.6, 160.3)
- added SW43: SW_Push, Button_Switch_Keyboard:SW_Cherry_MX_1.00u_PCB, F.Cu at (355.6, 150.8)
- added SW44: SW_Push, Button_Switch_Keyboard:SW_Cherry_MX_1.75u_PCB, F.Cu at (67.5, 169.9)
- added SW45: SW_Push, Button_Switch_Keyboard:SW_Cherry_MX_1.00u_PCB, F.Cu at (93.7, 169.9)
- added SW46: SW_Push, Button_Switch_Keyboard:SW_Cherry_MX_1.00u_PCB, F.Cu at (112.7, 169.9)
- added SW47: SW_Push, Button_Switch_Keyboard:SW_Cherry_MX_1.00u_PCB, F.Cu at (131.8, 169.9)
- added SW48: SW_Push, Button_Switch_Keyboard:SW_Cherry_MX_1.00u_PCB, F.Cu at (150.8, 169.9)
- added SW49: SW_Push, Button_Switch_Keyboard:SW_Cherry_MX_1.00u_PCB, F.Cu at (169.9, 169.9)
- added SW5: SW_Push, Button_Switch_Keyboard:SW_Cherry_MX_1.00u_PCB, F.Cu at (141.3, 108.0)
- added SW50: SW_Push, Button_Switch_Keyboard:SW_Cherry_MX_1.00u_PCB, F.Cu at (188.9, 169.9)
- added SW51: SW_Push, Button_Switch_Keyboard:SW_Cherry_MX_1.00u_PCB, F.Cu at (208.0, 169.9)
- added SW52: SW_Push, Button_Switch_Keyboard:SW_Cherry_MX_1.00u_PCB, F.Cu at (227.0, 169.9)
- added SW53: SW_Push, Button_Switch_Keyboard:SW_Cherry_MX_1.00u_PCB, F.Cu at (246.1, 169.9)
- added SW54: SW_Push, Button_Switch_Keyboard:SW_Cherry_MX_1.00u_PCB, F.Cu at (265.1, 169.9)
- added SW55: SW_Push, Button_Switch_Keyboard:SW_Cherry_MX_1.00u_PCB, F.Cu at (284.2, 169.9)
- added SW56: SW_Push, Button_Switch_Keyboard:SW_Cherry_MX_1.00u_PCB, F.Cu at (303.2, 169.9)
- added SW57: SW_Push, Button_Switch_Keyboard:SW_Cherry_MX_1.00u_PCB, F.Cu at (355.6, 169.9)
- added SW58: SW_Push, Button_Switch_Keyboard:SW_Cherry_MX_1.25u_PCB, F.Cu at (62.7, 188.9)
- added SW59: SW_Push, Button_Switch_Keyboard:SW_Cherry_MX_1.00u_PCB, F.Cu at (84.1, 188.9)
- added SW6: SW_Push, Button_Switch_Keyboard:SW_Cherry_MX_1.00u_PCB, F.Cu at (165.1, 108.0)
- added SW60: SW_Push, Button_Switch_Keyboard:SW_Cherry_MX_1.00u_PCB, F.Cu at (103.2, 188.9)
- added SW61: SW_Push, Button_Switch_Keyboard:SW_Cherry_MX_1.00u_PCB, F.Cu at (122.2, 188.9)
- added SW62: SW_Push, Button_Switch_Keyboard:SW_Cherry_MX_1.00u_PCB, F.Cu at (141.3, 188.9)
- added SW63: SW_Push, Button_Switch_Keyboard:SW_Cherry_MX_1.00u_PCB, F.Cu at (160.3, 188.9)
- added SW64: SW_Push, Button_Switch_Keyboard:SW_Cherry_MX_1.00u_PCB, F.Cu at (179.4, 188.9)
- added SW65: SW_Push, Button_Switch_Keyboard:SW_Cherry_MX_1.00u_PCB, F.Cu at (198.4, 188.9)
- added SW66: SW_Push, Button_Switch_Keyboard:SW_Cherry_MX_1.00u_PCB, F.Cu at (217.5, 188.9)
- added SW67: SW_Push, Button_Switch_Keyboard:SW_Cherry_MX_1.00u_PCB, F.Cu at (236.5, 188.9)
- added SW68: SW_Push, Button_Switch_Keyboard:SW_Cherry_MX_1.00u_PCB, F.Cu at (255.6, 188.9)
- added SW69: SW_Push, Button_Switch_Keyboard:SW_Cherry_MX_1.00u_PCB, F.Cu at (274.6, 188.9)
- added SW7: SW_Push, Button_Switch_Keyboard:SW_Cherry_MX_1.00u_PCB, F.Cu at (184.2, 108.0)
- added SW70: SW_Push, Button_Switch_Keyboard:SW_Cherry_MX_1.75u_PCB, F.Cu at (300.8, 188.9)
- added SW71: SW_Push, Button_Switch_Keyboard:SW_Cherry_MX_1.00u_PCB, F.Cu at (355.6, 188.9)
- added SW72: SW_Push, Button_Switch_Keyboard:SW_Cherry_MX_1.00u_PCB, F.Cu at (331.8, 193.7)
- added SW73: SW_Push, Button_Switch_Keyboard:SW_Cherry_MX_1.25u_PCB, F.Cu at (62.7, 208.0)
- added SW74: SW_Push, Button_Switch_Keyboard:SW_Cherry_MX_1.25u_PCB, F.Cu at (86.5, 208.0)
- added SW75: SW_Push, Button_Switch_Keyboard:SW_Cherry_MX_1.25u_PCB, F.Cu at (110.3, 208.0)
- added SW76: SW_Push, PCM_Switch_Keyboard_Cherry_MX:SW_Cherry_MX_PCB_6.25u, F.Cu at (179.2, 213.0)
- added SW77: SW_Push, Button_Switch_Keyboard:SW_Cherry_MX_1.00u_PCB, F.Cu at (250.8, 208.0)
- added SW78: SW_Push, Button_Switch_Keyboard:SW_Cherry_MX_1.00u_PCB, F.Cu at (269.9, 208.0)
- added SW79: SW_Push, Button_Switch_Keyboard:SW_Cherry_MX_1.00u_PCB, F.Cu at (288.9, 208.0)
- added SW8: SW_Push, Button_Switch_Keyboard:SW_Cherry_MX_1.00u_PCB, F.Cu at (203.2, 108.0)
- added SW80: SW_Push, Button_Switch_Keyboard:SW_Cherry_MX_1.00u_PCB, F.Cu at (312.7, 212.7)
- added SW81: SW_Push, Button_Switch_Keyboard:SW_Cherry_MX_1.00u_PCB, F.Cu at (331.8, 212.7)
- added SW82: SW_Push, Button_Switch_Keyboard:SW_Cherry_MX_1.00u_PCB, F.Cu at (350.8, 212.7)
- added SW9: SW_Push, Button_Switch_Keyboard:SW_Cherry_MX_1.00u_PCB, F.Cu at (222.2, 108.0)
- added TP1: BOOTSEL, TestPoint:TestPoint_Pad_D1.5mm, B.Cu at (221.7, 45.1)
- added TP11: VDD3, TestPoint:TestPoint_Pad_D1.5mm, B.Cu at (218.1, 52.2)
- added TP12: VDD18, TestPoint:TestPoint_Pad_D1.5mm, B.Cu at (214.6, 45.1)
- added TP13: VBUS_UP, TestPoint:TestPoint_Pad_D1.5mm, B.Cu at (214.6, 48.7)
- added TP14: GND, TestPoint:TestPoint_Pad_D1.5mm, B.Cu at (214.6, 52.2)
- added TP2: -RESET, TestPoint:TestPoint_Pad_D1.5mm, B.Cu at (221.7, 48.7)
- added TP3: 3V3, TestPoint:TestPoint_Pad_D1.5mm, B.Cu at (221.7, 52.2)
- added TP4: 5VUSB, TestPoint:TestPoint_Pad_D1.5mm, B.Cu at (218.1, 45.1)
- added TP5: GND, TestPoint:TestPoint_Pad_D1.5mm, B.Cu at (218.1, 48.7)
- added U1: RP2040_Stamp, RP2040 Stamp:RP2040_Stamp_THT, B.Cu at (192.6, 88.1)
- added U2: SL2.1A, SL2.1a:SOP-16_L10.0-W3.9-P1.27-LS6.0-BL, B.Cu at (328.6, 92.4)
- added Y1: 12MHz Crystal, Crystal:Crystal_SMD_3225-4Pin_3.2x2.5mm, B.Cu at (210.2, 45.6)
Routing:
- net USB3_D+: track 0.00 -> 36.5 mm
- net USB3_D-: track 0.00 -> 36.2 mm
- net VBUS_UP: track 0.00 -> 32.0 mm, vias 0 -> 2
- net Net-(D85-VP): track 0.00 -> 30.4 mm, vias 0 -> 2
- net Net-USB3-D-: track 0.00 -> 21.2 mm
- net USB_UP_D-: track 0.00 -> 20.2 mm
- net Net-J10-D-: track 0.00 -> 19.7 mm, vias 0 -> 2
- net Net-J10-D+: track 0.00 -> 19.5 mm, vias 0 -> 2
- net Net-USB3-D+: track 0.00 -> 18.7 mm
- net Net-(D86-VP): track 0.00 -> 18.1 mm
- net USB_UP_D+: track 0.00 -> 17.8 mm
- net USB2_D-: track 0.00 -> 13.8 mm, vias 0 -> 2
- net USB2_D+: track 0.00 -> 13.8 mm, vias 0 -> 2
- net USB4_D-: track 0.00 -> 12.4 mm
- net USB4_D+: track 0.00 -> 12.3 mm
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Other:
- board text added: "UPSTREAM"

Commit message: backup
Parts:
- moved FB3 151.6 mm to (367.3, 69.2), turned to 0 degrees
- moved FB2 143.2 mm to (331.5, 117.3)
- moved FB7 135.8 mm to (352.4, 72.8), turned to 0 degrees
- moved TP13 118.4 mm to (330.2, 74.1), turned to 0 degrees
- moved R9 99.9 mm to (371.5, 66.0), turned to -90 degrees
- moved R6 96.0 mm to (336.7, 114.6)
- moved C7 88.0 mm to (312.3, 75.9), turned to -90 degrees
- moved R2 87.9 mm to (336.6, 111.1)
- moved F1 87.2 mm to (320.0, 77.0), turned to 0 degrees
- moved R1 65.5 mm to (332.2, 69.1)
- moved R5 64.9 mm to (333.0, 65.7), turned to -90 degrees
- moved FB4 41.7 mm to (315.1, 77.0)
- moved FB1 33.5 mm to (319.1, 68.3), turned to -90 degrees
- moved R8 30.1 mm to (367.7, 65.0), turned to -90 degrees
- moved R13 0.78 mm to (351.6, 67.5)
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Connections:
- J1 pad 1: (no net) -> SHLD
- J1 pad 2: (no net) -> SHLD
Routing:
- net SHLD: track 9.44 -> 35.0 mm
- net VBUS_UP: track 32.0 -> 36.8 mm
- net Net-(F1-Pad1): track 0.00 -> 2.58 mm
- net +5V: track 0.00 -> 2.08 mm

Commit message: removed JST connectors for USBs
Parts:
- removed JP1: SolderJumper-Bridged, Jumper:SolderJumper-2_P1.3mm_Bridged_RoundedPad1.0x1.5mm
- removed Y1: 12MHz Crystal, Crystal:Crystal_SMD_3225-4Pin_3.2x2.5mm
- moved FB5 120.4 mm to (312.7, 110.3), turned to -90 degrees
- moved F2 113.6 mm to (314.9, 113.4)
- moved TP12 111.7 mm to (318.2, 87.0)
- moved C9 103.2 mm to (291.3, 79.4), turned to -90 degrees
- moved TP11 102.1 mm to (314.3, 86.2)
- moved C3 89.3 mm to (311.1, 87.8), turned to 90 degrees
- moved C1 86.3 mm to (315.4, 89.4), turned to 0 degrees
- moved C8 82.8 mm to (317.5, 109.5), turned to 0 degrees
- moved C2 82.2 mm to (319.2, 91.0), turned to -90 degrees
- moved R9 17.1 mm to (354.8, 69.7)
- moved D85 17.1 mm to (342.3, 88.0)
- moved R5 17.1 mm to (316.3, 69.4)
- moved C7 17.1 mm to (295.6, 79.6)
- moved D83 17.1 mm to (307.8, 87.2)
- moved D86 17.1 mm to (324.0, 90.4)
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Connections:
- net Net-J10-D+ renamed Net-(J10-D+)
- net Net-J10-D- renamed Net-(J10-D-)
- net Net-J6-D+ renamed Net-(J6-D+)
- net Net-J6-D- renamed Net-(J6-D-)
- net Net-U2-D+ renamed Net-(U2-DP)
- net Net-U2-D- renamed Net-(U2-DM)
- net Net-USB3-D+ renamed Net-(D85-L2-Pad3)
- net Net-USB3-D- renamed Net-(D85-L1-Pad1)
- C9 pad 1: +5V -> GND
- C9 pad 2: GND -> +5V
- J1 pad 1: SHLD -> (no net)
- J1 pad 2: SHLD -> (no net)
- J9 pad 2: SHLD -> (no net)
- U2 pad 15: Net-(U2-XOUT) -> unconnected-(U2-XOUT-Pad15)
- U2 pad 16: Net-(JP1-A) -> GND
Routing:
- net USB3_D+: track 36.5 -> 0.00 mm
- net USB3_D-: track 36.2 -> 0.00 mm
- net USB2_D-: track 13.8 -> 0.00 mm, vias 2 -> 0
- net USB2_D+: track 13.8 -> 0.00 mm, vias 2 -> 0
- net USB4_D-: track 12.4 -> 0.00 mm
- net USB4_D+: track 12.3 -> 0.00 mm
- net Net-(U2-VDD18): track 0.00 -> 10.5 mm
- net Net-(U2-VDD33): track 0.00 -> 9.31 mm
- net Net-(J6-D+): track 6.05 -> 0.00 mm
- net Net-(J6-D-): track 5.97 -> 0.00 mm
- net Net-(U2-DM): track 5.24 -> 0.00 mm
- net Net-(U2-DP): track 5.21 -> 0.00 mm
- net Net-(U2-VDD5): track 0.00 -> 4.76 mm
- net +5V: track 2.08 -> 6.49 mm
- net Net-(D84-VP): track 10.1 -> 14.0 mm
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Other:
- board outline added: 317.5 x 163.5 mm
