File: Quanta_v1/Quanta_v1.kicad_sch (KiCad schematic)
At the start: 236 parts, among them J1 USB_C_Receptacle_USB2.0, J10 USB_A_Receptacle_UBS2.0, J11 Conn_01x01_Socket GND, J12 Conn_01x06_Socket GPIOs, J13 Conn_01x01_Socket GPIO0, J2 Conn_01x02_Socket VBUS 5V, J3 Conn_01x02_Socket 3V3, J4 Conn_01x02_Socket VBAT, J5 Conn_01x04_Socket SWL, J6 USB_A_Receptacle_UBS2.0, J7 JSTConn USB3, J8 JSTConn USB4, J9 USB_C_Receptacle_USB2.0, SW1 SW_Push, SW10 SW_Push, SW11 SW_Push, SW12 SW_Push, SW13 SW_Push, SW14 SW_Push, SW15 SW_Push, SW16 SW_Push, SW17 SW_Push, SW18 SW_Push, SW19 SW_Push, SW2 SW_Push, SW20 SW_Push, SW21 SW_Push, SW22 SW_Push, SW23 SW_Push, SW24 SW_Push, SW25 SW_Push, SW26 SW_Push, SW27 SW_Push, SW28 SW_Push, SW29 SW_Push, SW3 SW_Push, SW30 SW_Push, SW31 SW_Push, SW32 SW_Push, SW33 SW_Push, SW34 SW_Push, SW35 SW_Push, SW36 SW_Push, SW37 SW_Push, SW38 SW_Push, SW39 SW_Push, SW4 SW_Push, SW40 SW_Push, SW41 SW_Push, SW42 SW_Push, SW43 SW_Push, SW44 SW_Push, SW45 SW_Push, SW46 SW_Push, SW47 SW_Push, SW48 SW_Push, SW49 SW_Push, SW5 SW_Push, SW50 SW_Push, SW51 SW_Push, SW52 SW_Push, SW53 SW_Push, SW54 SW_Push, SW55 SW_Push, SW56 SW_Push, SW57 SW_Push, SW58 SW_Push, SW59 SW_Push, SW6 SW_Push, SW60 SW_Push, SW61 SW_Push, SW62 SW_Push, SW63 SW_Push, SW64 SW_Push, SW65 SW_Push, SW66 SW_Push, SW67 SW_Push, SW68 SW_Push, SW69 SW_Push, SW7 SW_Push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

Commit message: start pcb
Parts:
- removed C5, C6, C8, C9: 100uF, symbol Device:C_Polarized
- removed R7: 2.7K, symbol Device:R
- removed TP10: EESDA, TestPoint:TestPoint_Pad_D1.5mm, symbol Connector:TestPoint
- removed TP6: LEDUSB1, TestPoint:TestPoint_Pad_D1.5mm, symbol Connector:TestPoint
- removed TP7: LEDUSB2, TestPoint:TestPoint_Pad_D1.5mm, symbol Connector:TestPoint
- removed TP8: LEDUSBDRV, TestPoint:TestPoint_Pad_D1.5mm, symbol Connector:TestPoint
- removed TP9: EESCL, TestPoint:TestPoint_Pad_D1.5mm, symbol Connector:TestPoint
- removed U3: FE1.1s, Package_SO:SSOP-28_3.9x9.9mm_P0.635mm, symbol Interface_USB:FE1.1s
- added C5, C6, C8, C9: 100uF, Capacitor_SMD:C_1206_3216Metric_Pad1.33x1.80mm_HandSolder, symbol Device:C_Small
- C1, C2, C4: footprint (none) -> Capacitor_SMD:C_0805_2012Metric_Pad1.18x1.45mm_HandSolder; JLCPCB (none) -> C380331
- C3, C7: footprint (none) -> Capacitor_SMD:C_0805_2012Metric_Pad1.18x1.45mm_HandSolder; JLCPCB (none) -> C784084
- D1: footprint Diode_THT:D_A-405_P7.62mm_Horizontal -> Diode_SMD:D_SOD-123; JLCPCB (none) -> C3018540
- D10, D11, D12, D13, D14, D15, D16, D17, D18, D19, D2, D20, D21, D22, D23, D24, D25, D26, D27, D28, D29, D3, D30, D31, D32, D33, D34, D35, D36, D37, D38, D39, D4, D40, D41, D42, D43, D44, D45, D46, D47, D48, D49, D5, D50, D51, D52, D53, D54, D55, D56, D57, D58, D59, D6, D60, D61, D62, D63, D64, D65, D66, D67, D68, D69, D7, D70, D71, D72, D73, D74, D75, D76, D77, D78, D79, D8, D80, D81, D82, D9: footprint Diode_THT:D_A-405_P7.62mm_Horizontal -> Diode_SMD:D_SOD-123
- D83, D84, D85, D86: footprint Package_TO_SOT_SMD_AKL:SOT-23-6 -> Package_TO_SOT_SMD:SOT-23-6_Handsoldering
- F1: footprint (none) -> Fuse:Fuse_1206_3216Metric_Pad1.42x1.75mm_HandSolder; JLCPCB (none) -> C140468
- F2: footprint (none) -> Fuse:Fuse_1206_3216Metric_Pad1.42x1.75mm_HandSolder; JLCPCB part numb (none) -> C468887
- F3, F4: footprint (none) -> Fuse:Fuse_1206_3216Metric_Pad1.42x1.75mm_HandSolder; JLCPCB (none) -> C468887
- FB4: footprint (none) -> PCM_Ferrite_SMD_Handsoldering_AKL:Ferrite_0603_1608Metric
- J1, J9: footprint (none) -> USB_C_socket_GT-USB-7010H:USB-C-SMD_G-SWITCH_GT-USB-7010EN; JLCPCB (none) -> C3001293
- J10: footprint (none) -> USB_A_horizontal_SMD_903-231A2031S10100:USB-A-SMD_903-231A2031S10100; JLCPCB (none) -> C42646
- J12: footprint (none) -> Connector_PinHeader_2.54mm:PinHeader_1x06_P2.54mm_Vertical
- J13: footprint (none) -> Connector_PinHeader_2.54mm:PinHeader_1x01_P2.54mm_Vertical
- J6: footprint (none) -> USB_A_vertical_KH-AF180ZJ-13.7:USB-A-TH_KH-AF180ZJ-13.7; JLCPCB (none) -> C2833345
- JP1: footprint (none) -> Jumper:SolderJumper-2_P1.3mm_Bridged_RoundedPad1.0x1.5mm
- R1, R12, R2, R8: footprint (none) -> Resistor_SMD:R_1206_3216Metric_Pad1.30x1.75mm_HandSolder; JLCPCB (none) -> C1021510
- R10, R11: footprint (none) -> Resistor_SMD:R_0603_1608Metric_Pad0.98x0.95mm_HandSolder; JLCPCB (none) -> C432813
- R13, R5, R6, R9: footprint (none) -> Resistor_SMD:R_0805_2012Metric_Pad1.20x1.40mm_HandSolder; JLCPCB (none) -> C163969
- R3, R4: footprint (none) -> Resistor_SMD:R_0603_1608Metric_Pad0.98x0.95mm_HandSolder; JLCPCB (none) -> C178023
- RED1: renamed from DSWRE1; footprint Diode_THT:D_A-405_P7.62mm_Horizontal -> Diode_SMD:D_SOD-123
- SW28: footprint Button_Switch_Keyboard:SW_Cherry_MX_1.50u_PCB -> Button_Switch_Keyboard:SW_Cherry_MX_1.00u_PCB
- SW29: footprint Button_Switch_Keyboard:SW_Cherry_MX_1.00u_PCB -> Button_Switch_Keyboard:SW_Cherry_MX_1.50u_PCB
- SW76: footprint Button_Switch_Keyboard:SW_Cherry_MX_6.25u_PCB -> PCM_Switch_Keyboard_Cherry_MX:SW_Cherry_MX_PCB_6.25u
- U1: footprint RP2040_Stamp:RP2040_Stamp_THT -> RP2040 Stamp:RP2040_Stamp_THT
- U2: footprint SL2:SOP-16_L10.0-W3.9-P1.27-LS6.0-BL -> SL2.1a:SOP-16_L10.0-W3.9-P1.27-LS6.0-BL
- renumbered SWRE1 to RESW1
Connections:
- net Column1: now also D1.1 (K), D14.1 (K), D29.1 (K), D44.1 (K), D58.1 (K), D73.1 (K); no longer D1.2 (A), D14.2 (A), D28.2 (A), D44.2 (A), D58.2 (A), D73.2 (A)
- net Column10: now also D10.1 (K), D23.1 (K), D38.1 (K), D53.1 (K), D67.1 (K), D77.1 (K); no longer D10.2 (A), D23.2 (A), D38.2 (A), D53.2 (A), D67.2 (A), D77.2 (A)
- net Column11: now also D11.1 (K), D24.1 (K), D39.1 (K), D54.1 (K), D68.1 (K), D78.1 (K); no longer D11.2 (A), D24.2 (A), D39.2 (A), D54.2 (A), D68.2 (A), D78.2 (A)
- net Column12: now also D12.1 (K), D25.1 (K), D40.1 (K), D55.1 (K), D69.1 (K), D79.1 (K); no longer D12.2 (A), D25.2 (A), D40.2 (A), D55.2 (A), D69.2 (A), D79.2 (A)
- net Column13: now also D13.1 (K), D26.1 (K), D41.1 (K), D56.1 (K), D70.1 (K), D80.1 (K); no longer D13.2 (A), D26.2 (A), D41.2 (A), D56.2 (A), D70.2 (A), D80.2 (A)
- net Column14: now also D27.1 (K), D42.1 (K), D71.1 (K), D81.1 (K); no longer D27.2 (A), D42.2 (A), D71.2 (A), D81.2 (A)
- net Column15: now also D28.1 (K), D43.1 (K), D57.1 (K), D72.1 (K), D82.1 (K), RED1.1 (K); no longer D29.2 (A), D43.2 (A), D57.2 (A), D72.2 (A), D82.2 (A), RED1.2 (A)
- net Column2: now also D15.1 (K), D2.1 (K), D30.1 (K), D45.1 (K), D59.1 (K), D74.1 (K); no longer D15.2 (A), D2.2 (A), D30.2 (A), D45.2 (A), D59.2 (A), D74.2 (A)
- net Column3: now also D16.1 (K), D3.1 (K), D31.1 (K), D46.1 (K), D60.1 (K), D75.1 (K); no longer D16.2 (A), D3.2 (A), D31.2 (A), D46.2 (A), D60.2 (A), D75.2 (A)
- net Column4: now also D17.1 (K), D32.1 (K), D4.1 (K), D47.1 (K), D61.1 (K); no longer D17.2 (A), D32.2 (A), D4.2 (A), D47.2 (A), D61.2 (A)
- net Column5: now also D18.1 (K), D33.1 (K), D48.1 (K), D5.1 (K), D62.1 (K); no longer D18.2 (A), D33.2 (A), D48.2 (A), D5.2 (A), D62.2 (A)
- net Column6: now also D19.1 (K), D34.1 (K), D49.1 (K), D6.1 (K), D63.1 (K); no longer D19.2 (A), D34.2 (A), D49.2 (A), D6.2 (A), D63.2 (A)
- net Column7: now also D20.1 (K), D35.1 (K), D50.1 (K), D64.1 (K), D7.1 (K), D76.1 (K); no longer D20.2 (A), D35.2 (A), D50.2 (A), D64.2 (A), D7.2 (A), D76.2 (A)
- net Column8: now also D21.1 (K), D36.1 (K), D51.1 (K), D65.1 (K), D8.1 (K); no longer D21.2 (A), D36.2 (A), D51.2 (A), D65.2 (A), D8.2 (A)
- net Column9: now also D22.1 (K), D37.1 (K), D52.1 (K), D66.1 (K), D9.1 (K); no longer D22.2 (A), D37.2 (A), D52.2 (A), D66.2 (A), D9.2 (A)
- net Row2: now also SW28.2; no longer SW29.2
- net Row3: now also SW29.2; no longer SW28.2
- net at SW10.1: now also D10.2 (A); no longer D10.1 (K)
- net at SW8.1: now also D8.2 (A); no longer D8.1 (K)
- net at SW43.1: now also D43.2 (A); no longer D43.1 (K)
- net at SW47.1: now also D47.2 (A); no longer D47.1 (K)
- net at SW72.1: now also D72.2 (A); no longer D72.1 (K)
- net at SW14.1: now also D14.2 (A); no longer D14.1 (K)
- net at SW39.1: now also D39.2 (A); no longer D39.1 (K)
- net at SW76.1: now also D76.2 (A); no longer D76.1 (K)
- net at SW59.1: now also D59.2 (A); no longer D59.1 (K)
- net at SW49.1: now also D49.2 (A); no longer D49.1 (K)
- net at SW63.1: now also D63.2 (A); no longer D63.1 (K)
- net at SW46.1: now also D46.2 (A); no longer D46.1 (K)
- net at SW20.1: now also D20.2 (A); no longer D20.1 (K)
- net at SW65.1: now also D65.2 (A); no longer D65.1 (K)
- net at SW38.1: now also D38.2 (A); no longer D38.1 (K)
- net at SW51.1: now also D51.2 (A); no longer D51.1 (K)
- net at D84.5 (VP), F2.1, J6.1 (VBUS): now also C8.2
- net at SW41.1: now also D41.2 (A); no longer D41.1 (K)
- net at SW52.1: now also D52.2 (A); no longer D52.1 (K)
- net at SW81.1: now also D81.2 (A); no longer D81.1 (K)
- net at SW42.1: now also D42.2 (A); no longer D42.1 (K)
- net at SW24.1: now also D24.2 (A); no longer D24.1 (K)
- net at SW33.1: now also D33.2 (A); no longer D33.1 (K)
- net at SW74.1: now also D74.2 (A); no longer D74.1 (K)
- net at SW71.1: now also D71.2 (A); no longer D71.1 (K)
- net at SW2.1: now also D2.2 (A); no longer D2.1 (K)
- net at SW44.1: now also D44.2 (A); no longer D44.1 (K)
- net at SW28.1: now also D28.2 (A); no longer D28.1 (K)
- net at SW32.1: now also D32.2 (A); no longer D32.1 (K)
- net at D85.5 (VP), F3.1, J9.A4 (VBUS)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: now also C5.1
- net at SW18.1: now also D18.2 (A); no longer D18.1 (K)
- net at SW12.1: now also D12.2 (A); no longer D12.1 (K)
- net at SW79.1: now also D79.2 (A); no longer D79.1 (K)
- net at SW13.1: now also D13.2 (A); no longer D13.1 (K)
- net at SW21.1: now also D21.2 (A); no longer D21.1 (K)
- net at SW64.1: now also D64.2 (A); no longer D64.1 (K)
- net at SW60.1: now also D60.2 (A); no longer D60.1 (K)
- net at SW78.1: now also D78.2 (A); no longer D78.1 (K)
- net at D86.5 (VP), F4.1, J10.1 (VBUS): now also C6.2
- net at SW50.1: now also D50.2 (A); no longer D50.1 (K)
- net at SW16.1: now also D16.2 (A); no longer D16.1 (K)
- net at SW48.1: now also D48.2 (A); no longer D48.1 (K)
- net at SW73.1: now also D73.2 (A); no longer D73.1 (K)
- net at SW75.1: now also D75.2 (A); no longer D75.1 (K)
- net at SW23.1: now also D23.2 (A); no longer D23.1 (K)
- net at SW68.1: now also D68.2 (A); no longer D68.1 (K)
- net at RESW1.S1: now also RED1.2 (A); no longer RED1.1 (K)
- net at SW61.1: now also D61.2 (A); no longer D61.1 (K)
- net at SW26.1: now also D26.2 (A); no longer D26.1 (K)
- net at SW45.1: now also D45.2 (A); no longer D45.1 (K)
- net at SW25.1: now also D25.2 (A); no longer D25.1 (K)
- net at SW58.1: now also D58.2 (A); no longer D58.1 (K)
- net at SW80.1: now also D80.2 (A); no longer D80.1 (K)
- net at SW29.1: now also D29.2 (A); no longer D29.1 (K)
- net at SW15.1: now also D15.2 (A); no longer D15.1 (K)
- net at SW82.1: now also D82.2 (A); no longer D82.1 (K)
- net at SW56.1: now also D56.2 (A); no longer D56.1 (K)
- net at SW77.1: now also D77.2 (A); no longer D77.1 (K)
- net at SW27.1: now also D27.2 (A); no longer D27.1 (K)
- net at SW31.1: now also D31.2 (A); no longer D31.1 (K)
- net at SW9.1: now also D9.2 (A); no longer D9.1 (K)
- net at SW70.1: now also D70.2 (A); no longer D70.1 (K)
- net at SW30.1: now also D30.2 (A); no longer D30.1 (K)
- net at SW66.1: now also D66.2 (A); no longer D66.1 (K)
- net at SW1.1: now also D1.2 (A); no longer D1.1 (K)
- net at SW17.1: now also D17.2 (A); no longer D17.1 (K)
- net at SW11.1: now also D11.2 (A); no longer D11.1 (K)
- net at SW62.1: now also D62.2 (A); no longer D62.1 (K)
- net at SW3.1: now also D3.2 (A); no longer D3.1 (K)
- net at SW19.1: now also D19.2 (A); no longer D19.1 (K)
- net at SW69.1: now also D69.2 (A); no longer D69.1 (K)
- net at SW54.1: now also D54.2 (A); no longer D54.1 (K)
- net at SW53.1: now also D53.2 (A); no longer D53.1 (K)
- net at SW36.1: now also D36.2 (A); no longer D36.1 (K)
- net at SW55.1: now also D55.2 (A); no longer D55.1 (K)
- net at SW34.1: now also D34.2 (A); no longer D34.1 (K)
- net at SW6.1: now also D6.2 (A); no longer D6.1 (K)
- net at SW7.1: now also D7.2 (A); no longer D7.1 (K)
- net at SW67.1: now also D67.2 (A); no longer D67.1 (K)
- net at SW35.1: now also D35.2 (A); no longer D35.1 (K)
- net at SW22.1: now also D22.2 (A); no longer D22.1 (K)
- net at SW57.1: now also D57.2 (A); no longer D57.1 (K)
- net at SW40.1: now also D40.2 (A); no longer D40.1 (K)
- net at SW4.1: now also D4.2 (A); no longer D4.1 (K)
- net at SW37.1: now also D37.2 (A); no longer D37.1 (K)
- net at SW5.1: now also D5.2 (A); no longer D5.1 (K)
- net +3V3 renamed GND
- net GND: now also C5.2, C6.1, C8.1, C9.2; no longer C3.2, C4.2, C7.2, D83.5 (VP), F1.2, FB4.2, FB5.1, FB6.1, FB8.1, J1.A4 (VBUS), J1.A9 (VBUS), J1.B4 (VBUS), J1.B9 (VBUS), J2.1 (Pin_1), J4.1 (Pin_1), R10.1, R11.1, TP13.1, TP4.1, U1.32 (VBAT), U1.33 (5V)
- new net +5V: C3.2, C7.2, C9.1, FB4.2, FB5.1, FB6.1, FB8.1, J2.1 (Pin_1), R10.1, R11.1, TP4.1, U1.33 (5V)
- new net VBAT: J4.1 (Pin_1), U1.32 (VBAT)
- new net VBUS_UP: C4.2, D83.5 (VP), F1.2, J1.A4 (VBUS), J1.A9 (VBUS), J1.B4 (VBUS), J1.B9 (VBUS), TP13.1
- no-connect marks 17 -> 4
Other:
- note removed: "old USB Hub deprecated"
- moved on the sheet: C4, C7, D1, D10, D11, D12, D13, D14, D15, D16, D17, D18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

Commit message: removed JST connectors for USBs
Parts:
- removed J7: JSTConn USB3, Connector_JST:JST_EH_S4B-EH_1x04_P2.50mm_Horizontal, symbol Connector_Generic:Conn_01x04
- removed J8: JSTConn USB4, Connector_JST:JST_EH_S4B-EH_1x04_P2.50mm_Horizontal, symbol Connector_Generic:Conn_01x04
- removed JP1: SolderJumper-Bridged, Jumper:SolderJumper-2_P1.3mm_Bridged_RoundedPad1.0x1.5mm, symbol Jumper:SolderJumper_2_Bridged
- removed Y1: 12MHz Crystal, Crystal:Crystal_SMD_3225-4Pin_3.2x2.5mm, symbol Device:Crystal
Connections:
- net +5V: now also C9.2; no longer C9.1
- net GND: now also C9.1, U2.16 (XIN); no longer C9.2
- no-connect marks 4 -> 5
Other:
- note removed: "Additional USB JST connectors"
- moved on the sheet: C9
