File: Quanta_RP2040Stamp/Quanta_RP2040Stamp.kicad_pcb (KiCad board)
At the start: 2 copper layers, 317.5 x 163.5 mm, 228 parts, among them J1 USB_C_Receptacle_USB2.0, J10 USB_A_Receptacle_UBS2.0, J11 Conn_01x01_Socket GND, J12 Conn_01x06_Socket GPIOs, J13 Conn_01x01_Socket GPIO0, J2 Conn_01x02_Socket VBUS 5V, J3 Conn_01x02_Socket 3V3, J4 Conn_01x02_Socket VBAT, J5 Conn_01x04_Socket SWL, J6 USB_A_Receptacle_UBS2.0, J7 JSTConn USB3, J8 JSTConn USB4, J9 USB_C_Receptacle_USB2.0, SW1 SW_Push, SW10 SW_Push, SW11 SW_Push, SW12 SW_Push, SW13 SW_Push, SW14 SW_Push, SW15 SW_Push, SW16 SW_Push, SW17 SW_Push, SW18 SW_Push, SW19 SW_Push, SW2 SW_Push, SW20 SW_Push, SW21 SW_Push, SW22 SW_Push, SW23 SW_Push, SW24 SW_Push, SW25 SW_Push, SW26 SW_Push, SW27 SW_Push, SW28 SW_Push, SW29 SW_Push, SW3 SW_Push, SW30 SW_Push, SW31 SW_Push, SW32 SW_Push, SW33 SW_Push, SW34 SW_Push, SW35 SW_Push, SW36 SW_Push, SW37 SW_Push, SW38 SW_Push, SW39 SW_Push, SW4 SW_Push, SW40 SW_Push, SW41 SW_Push, SW42 SW_Push, SW43 SW_Push, SW44 SW_Push, SW45 SW_Push, SW46 SW_Push, SW47 SW_Push, SW48 SW_Push, SW49 SW_Push, SW5 SW_Push, SW50 SW_Push, SW51 SW_Push, SW52 SW_Push, SW53 SW_Push, SW54 SW_Push, SW55 SW_Push, SW56 SW_Push, SW57 SW_Push, SW58 SW_Push, SW59 SW_Push, SW6 SW_Push, SW60 SW_Push, SW61 SW_Push, SW62 SW_Push, SW63 SW_Push, SW64 SW_Push, SW65 SW_Push, SW66 SW_Push, SW67 SW_Push, SW68 SW_Push, SW69 SW_Push, SW7 SW_Push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

Commit message: rename kicad project
Parts:
- removed J7: JSTConn USB3, Connector_JST:JST_EH_S4B-EH_1x04_P2.50mm_Horizontal
- removed J8: JSTConn USB4, Connector_JST:JST_EH_S4B-EH_1x04_P2.50mm_Horizontal
- moved FB6 127.0 mm to (337.3, 86.5), turned to 90 degrees
- moved FB8 119.2 mm to (331.4, 86.8), turned to 90 degrees
- moved C4 101.7 mm to (298.2, 78.3), turned to 0 degrees
- moved J5 92.7 mm to (213.5, 98.2), turned to 0 degrees
- moved J11 92.4 mm to (181.8, 69.8), turned to -90 degrees
- moved TP14 85.4 mm to (296.7, 75.5), turned to -90 degrees
- moved F4 77.6 mm to (329.4, 83.3), turned to 0 degrees
- moved C6 74.9 mm to (319.8, 80.4), turned to 0 degrees
- moved TP4 73.4 mm to (282.2, 81.0), turned to 0 degrees
- moved J13 73.3 mm to (208.8, 100.4)
- moved R11 73.2 mm to (345.4, 74.6), turned to 90 degrees
- moved F3 73.0 mm to (337.3, 82.1), turned to -90 degrees
- moved R10 70.8 mm to (342.4, 73.9), turned to 90 degrees
- moved TP1 52.5 mm to (208.5, 96.0), turned to -90 degrees
- moved TP2 46.5 mm to (208.4, 93.3), turned to -90 degrees
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Connections:
- FB1 pad 1: SHLD -> Net-(J1-SHIELD)
- FB2 pad 1: SHLD -> Net-(J6-Shield)
- FB3 pad 1: SHLD -> Net-(J9-SHIELD)
- FB7 pad 1: SHLD -> Net-(J10-Shield)
- J10 pad 5: SHLD -> Net-(J10-Shield)
- J6 pad 5: SHLD -> Net-(J6-Shield)
- R1 pad 2: SHLD -> Net-(J1-SHIELD)
- R12 pad 2: SHLD -> Net-(J10-Shield)
- R13 pad 2: SHLD -> Net-(J10-Shield)
- R2 pad 2: SHLD -> Net-(J6-Shield)
- R5 pad 2: SHLD -> Net-(J1-SHIELD)
- R6 pad 2: SHLD -> Net-(J6-Shield)
- R8 pad 2: SHLD -> Net-(J9-SHIELD)
- R9 pad 2: SHLD -> Net-(J9-SHIELD)
- SW76 pad 1: Net-(D76-A) -> Row6
- SW76 pad 2: Row6 -> Net-(D76-A)
- U1 pad 10: Column3 -> Column7
- U1 pad 11: Column4 -> Column6
- U1 pad 13: Column6 -> Column4
- U1 pad 14: Column7 -> Column3
- U1 pad 15: Column8 -> Column2
- U1 pad 16: Column9 -> Column1
- U1 pad 17: Column10 -> Row1
- U1 pad 18: Column11 -> Row2
- U1 pad 19: Column12 -> Row3
- U1 pad 2: Row1 -> Column15
- U1 pad 20: Column13 -> Row4
- U1 pad 21: Column14 -> Row5
- U1 pad 22: Column15 -> Row6
- U1 pad 3: Row2 -> Column14
- U1 pad 4: Row3 -> Column13
- U1 pad 5: Row4 -> Column12
- U1 pad 6: Row5 -> Column11
- U1 pad 7: Row6 -> Column10
- U1 pad 8: Column1 -> Column9
- U1 pad 9: Column2 -> Column8
Routing:
- net +5V: track 6.49 -> 93.2 mm, vias 0 -> 6
- net SHLD: track 37.4 -> 0.00 mm
- net +3.3V: track 0.00 -> 25.2 mm
- net Net-(J6-Shield): track 0.00 -> 12.9 mm
- net VBAT: track 0.00 -> 12.3 mm
- net Net-(J5-Pin_2): track 0.00 -> 11.1 mm
- net Net-(J5-Pin_3): track 0.00 -> 10.8 mm
- net Net-(J9-SHIELD): track 0.00 -> 10.3 mm
- net Net-(D56-A): track 0.00 -> 9.43 mm
- net Net-(D40-A): track 0.00 -> 9.43 mm
- net Net-(D24-A): track 0.00 -> 9.43 mm
- net Net-(D22-A): track 0.00 -> 9.43 mm
- net Net-(D19-A): track 0.00 -> 9.43 mm
- net Net-(D13-A): track 0.00 -> 9.43 mm
- net Net-(D82-A): track 0.00 -> 9.43 mm
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Other:
- outline, holes or cut-outs redrawn
- board text added: "Place RP2040 Stamp here"
