File: Quanta_RP2040Stamp/Quanta_RP2040Stamp.kicad_sch (KiCad schematic)
At the start: 225 parts, among them J1 USB_C_Receptacle_USB2.0, J10 USB_A_Receptacle_UBS2.0, J11 Conn_01x01_Socket GND, J12 Conn_01x06_Socket GPIOs, J13 Conn_01x01_Socket GPIO0, J2 Conn_01x02_Socket VBUS 5V, J3 Conn_01x02_Socket 3V3, J4 Conn_01x02_Socket VBAT, J5 Conn_01x04_Socket SWL, J6 USB_A_Receptacle_UBS2.0, J9 USB_C_Receptacle_USB2.0, SW1 SW_Push, SW10 SW_Push, SW11 SW_Push, SW12 SW_Push, SW13 SW_Push, SW14 SW_Push, SW15 SW_Push, SW16 SW_Push, SW17 SW_Push, SW18 SW_Push, SW19 SW_Push, SW2 SW_Push, SW20 SW_Push, SW21 SW_Push, SW22 SW_Push, SW23 SW_Push, SW24 SW_Push, SW25 SW_Push, SW26 SW_Push, SW27 SW_Push, SW28 SW_Push, SW29 SW_Push, SW3 SW_Push, SW30 SW_Push, SW31 SW_Push, SW32 SW_Push, SW33 SW_Push, SW34 SW_Push, SW35 SW_Push, SW36 SW_Push, SW37 SW_Push, SW38 SW_Push, SW39 SW_Push, SW4 SW_Push, SW40 SW_Push, SW41 SW_Push, SW42 SW_Push, SW43 SW_Push, SW44 SW_Push, SW45 SW_Push, SW46 SW_Push, SW47 SW_Push, SW48 SW_Push, SW49 SW_Push, SW5 SW_Push, SW50 SW_Push, SW51 SW_Push, SW52 SW_Push, SW53 SW_Push, SW54 SW_Push, SW55 SW_Push, SW56 SW_Push, SW57 SW_Push, SW58 SW_Push, SW59 SW_Push, SW6 SW_Push, SW60 SW_Push, SW61 SW_Push, SW62 SW_Push, SW63 SW_Push, SW64 SW_Push, SW65 SW_Push, SW66 SW_Push, SW67 SW_Push, SW68 SW_Push, SW69 SW_Push, SW7 SW_Push, SW70 SW_Push, SW71 SW_Push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

Commit message: rename kicad project
Connections:
- net Column1: now also U1.16 (GPIO15); no longer U1.8 (GPIO7)
- net Column10: now also U1.7 (GPIO6); no longer U1.17 (GPIO16)
- net Column11: now also U1.6 (GPIO5); no longer U1.18 (GPIO17)
- net Column12: now also U1.5 (GPIO4); no longer U1.19 (GPIO18)
- net Column13: now also U1.4 (GPIO3); no longer U1.20 (GPIO19)
- net Column14: now also U1.3 (GPIO2); no longer U1.21 (GPIO20)
- net Column15: now also U1.2 (GPIO1); no longer U1.22 (GPIO21)
- net Column2: now also U1.15 (GPIO14); no longer U1.9 (GPIO8)
- net Column3: now also U1.14 (GPIO13); no longer U1.10 (GPIO9)
- net Column4: now also U1.13 (GPIO12); no longer U1.11 (GPIO10)
- net Column6: now also U1.11 (GPIO10); no longer U1.13 (GPIO12)
- net Column7: now also U1.10 (GPIO9); no longer U1.14 (GPIO13)
- net Column8: now also U1.9 (GPIO8); no longer U1.15 (GPIO14)
- net Column9: now also U1.8 (GPIO7); no longer U1.16 (GPIO15)
- net Row1: now also U1.17 (GPIO16); no longer U1.2 (GPIO1)
- net Row2: now also U1.18 (GPIO17); no longer U1.3 (GPIO2)
- net Row3: now also U1.19 (GPIO18); no longer U1.4 (GPIO3)
- net Row4: now also U1.20 (GPIO19); no longer U1.5 (GPIO4)
- net Row5: now also U1.21 (GPIO20); no longer U1.6 (GPIO5)
- net Row6: now also SW76.1, U1.22 (GPIO21); no longer SW76.2, U1.7 (GPIO6)
- net at D76.2 (A): now also SW76.2; no longer SW76.1
- removed net SHLD: FB1.1, FB2.1, FB3.1, FB7.1, J1.S1 (SHIELD), J10.5 (Shield), J6.5 (Shield), J9.S1 (SHIELD), R1.2, R12.2, R13.2, R2.2, R5.2, R6.2, R8.2, R9.2
- new net: FB2.1, J6.5 (Shield), R2.2, R6.2
- new net: FB1.1, J1.S1 (SHIELD), R1.2, R5.2
- new net: FB7.1, J10.5 (Shield), R12.2, R13.2
- new net: FB3.1, J9.S1 (SHIELD), R8.2, R9.2
Other:
- title: Quanta Keyboard Schematic -> Quanta Keyboard Schematic (RP2040 Stamp)
- moved on the sheet: SW76
