File: Quanta_RP2040Stamp_JLCPCBAoptimized/Quanta_RP2040Stamp_JLCPCBAoptimized.kicad_sch (KiCad schematic)
At the start: 218 parts, among them J1 USB_C_Receptacle_USB2.0, J10 USB_A_Receptacle_UBS2.0, J11 Conn_01x01_Socket GND, J12 Conn_01x06_Socket GPIOs, J13 Conn_01x01_Socket GPIO0, J2 Conn_01x02_Socket VBUS 5V, J3 Conn_01x02_Socket 3V3, J4 Conn_01x02_Socket VBAT, J5 Conn_01x04_Socket SWL, J6 USB_A_Receptacle_UBS2.0, J9 USB_C_Receptacle_USB2.0, SW1 SW_Push, SW10 SW_Push, SW11 SW_Push, SW12 SW_Push, SW13 SW_Push, SW14 SW_Push, SW15 SW_Push, SW16 SW_Push, SW17 SW_Push, SW18 SW_Push, SW19 SW_Push, SW2 SW_Push, SW20 SW_Push, SW21 SW_Push, SW22 SW_Push, SW23 SW_Push, SW24 SW_Push, SW25 SW_Push, SW26 SW_Push, SW27 SW_Push, SW28 SW_Push, SW29 SW_Push, SW3 SW_Push, SW30 SW_Push, SW31 SW_Push, SW32 SW_Push, SW33 SW_Push, SW34 SW_Push, SW35 SW_Push, SW36 SW_Push, SW37 SW_Push, SW38 SW_Push, SW39 SW_Push, SW4 SW_Push, SW40 SW_Push, SW41 SW_Push, SW42 SW_Push, SW43 SW_Push, SW44 SW_Push, SW45 SW_Push, SW46 SW_Push, SW47 SW_Push, SW48 SW_Push, SW49 SW_Push, SW5 SW_Push, SW50 SW_Push, SW51 SW_Push, SW52 SW_Push, SW53 SW_Push, SW54 SW_Push, SW55 SW_Push, SW56 SW_Push, SW57 SW_Push, SW58 SW_Push, SW59 SW_Push, SW6 SW_Push, SW60 SW_Push, SW61 SW_Push, SW62 SW_Push, SW63 SW_Push, SW64 SW_Push, SW65 SW_Push, SW66 SW_Push, SW67 SW_Push, SW68 SW_Push, SW69 SW_Push, SW7 SW_Push, SW70 SW_Push, SW71 SW_Push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

Commit message: update rev of optimized pcb
Parts:
- removed FB7: 600R, PCM_Ferrite_SMD_Handsoldering_AKL:Ferrite_0805_2012Metric, symbol Device:FerriteBead
- removed FB8: 600R 500mA, PCM_Ferrite_SMD_Handsoldering_AKL:Ferrite_0805_2012Metric, symbol Device:FerriteBead_Small
- removed J10: USB_A_Receptacle_UBS2.0, USB_A_horizontal_SMD_903-231A2031S10100:USB-A-SMD_903-231A2031S10100, symbol Connector:USB_A
- removed J12: Conn_01x06_Socket GPIOs, Connector_PinHeader_2.54mm:PinHeader_1x06_P2.54mm_Vertical, symbol Connector:Conn_01x06_Socket
- added FB7: 600R 500mA, PCM_Ferrite_SMD_Handsoldering_AKL:Ferrite_0805_2012Metric, symbol Device:FerriteBead_Small
- added FB8: 600R, PCM_Ferrite_SMD_Handsoldering_AKL:Ferrite_0805_2012Metric, symbol Device:FerriteBead
- added J7: USB_C_Receptacle_USB2.0, USB_C_socket_GT-USB-7010H:USB-C-SMD_G-SWITCH_GT-USB-7010EN, symbol Connector:USB_C_Receptacle_USB2.0
- added J8: Conn_01x04_Socket I2C display, Connector_PinHeader_2.54mm:PinHeader_1x04_P2.54mm_Vertical, symbol Connector:Conn_01x04_Socket
- added R5, R8: 43k, Resistor_SMD:R_0603_1608Metric_Pad0.98x0.95mm_HandSolder, symbol Device:R_Small
- added R6, R9: 15k, Resistor_SMD:R_0603_1608Metric_Pad0.98x0.95mm_HandSolder, symbol Device:R_Small
- D1: JLCPCB C3018540 -> C81598
- J5: value Conn_01x04_Socket SWL -> Conn_01x04_Socket SWD
- RESW1: footprint Rotary_Encoder:RotaryEncoder_Bourns_Vertical_PEC12R-3xxxF-Sxxxx -> PEC12R-4120F-S0012:SW-TH_PEC12R-4120F-S0012
Connections:
- net +3.3V: now also J8.2 (Pin_2)
- net +5V: now also FB7.1, R6.2, R9.2
- net GND: now also C6.2, FB8.1, J7.A1 (GND), J7.A12 (GND), J7.B1 (GND), J7.B12 (GND), J8.1 (Pin_1); no longer C6.1
- net USB1_D+: now also U2.4 (DP3); no longer U2.8 (DP1)
- net USB1_D-: now also U2.3 (DM3); no longer U2.7 (DM1)
- net USB2_D+: now also U2.2 (DP4); no longer U2.6 (DP2)
- net USB2_D-: now also U2.1 (DM4); no longer U2.5 (DM2)
- net USB3_D+: now also U2.8 (DP1); no longer U2.4 (DP3)
- net USB3_D-: now also U2.7 (DM1); no longer U2.3 (DM3)
- net USB4_D+: now also D86.4 (L2), U2.6 (DP2); no longer D86.6 (L1), U2.2 (DP4)
- net USB4_D-: now also D86.6 (L1), U2.5 (DM2); no longer D86.4 (L2), U2.1 (DM4)
- net at D86.5 (VP): now also C6.1, FB7.2, J7.A4 (VBUS), J7.A9 (VBUS), J7.B4 (VBUS), J7.B9 (VBUS); no longer C6.2
- net I2C1-SDA: now reaches U1.27 (GPIO26)
- net I2C1-SDA: now also J8.4 (Pin_4)
- net I2C1-SCL: now reaches U1.28 (GPIO27)
- net I2C1-SCL: now also J8.3 (Pin_3)
- net at D86.1 (L1): now also J7.A7 (D-), J7.B7 (D-)
- net at D86.3 (L2): now also J7.A6 (D+), J7.B6 (D+)
- new net: R5.2, R6.1
- new net: R8.2, R9.1
- new net: J7.A5 (CC1), R5.1
- new net: J7.B5 (CC2), R8.1
- new net: FB8.2, J7.S1 (SHIELD)
- no-connect marks 5 -> 7
Other:
- note added: "Downstream USB C socket (USB 4)"
- note added: "OLED I2C display connector"
- note removed: "Downstream USB A socket (USB 4)"
- moved on the sheet: TP13

Commit message: routed matrix for optimized version
Parts:
- removed J11: Conn_01x01_Socket GND, Connector_PinHeader_2.54mm:PinHeader_1x01_P2.54mm_Vertical, symbol Connector:Conn_01x01_Socket
- added J10: Conn_01x05_Socket GPIOs, Connector_PinHeader_2.54mm:PinHeader_1x05_P2.54mm_Vertical, symbol Connector:Conn_01x05_Socket
Connections:
- net GND: now also J10.5 (Pin_5)
- net USBUP+: now reaches D83.4 (L2), U2.10 (DP)
- net USBUP-: now reaches D83.6 (L1), U2.9 (DM)
- net USB2+: now reaches D84.1 (L1), J6.3 (D+)
- net USB2-: now reaches D84.3 (L2), J6.2 (D-)
- net USB3-: now reaches D85.1 (L1), J9.A7 (D-), J9.B7 (D-)
- net USB3+: now reaches D85.3 (L2), J9.A6 (D+), J9.B6 (D+)
- net at U1.25 (GPIO24): now also J10.1 (Pin_1)
- net at U1.26 (GPIO25): now also J10.2 (Pin_2)
- net at U1.29 (GPIO28): now also J10.3 (Pin_3)
- net at U1.30 (GPIO29): now also J10.4 (Pin_4)
- net USB4-: now reaches D86.1 (L1), J7.A7 (D-), J7.B7 (D-)
- net USB4+: now reaches D86.3 (L2), J7.A6 (D+), J7.B6 (D+)
Other:
- moved on the sheet: TP5
Changed lines of the file:
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@@
   (junction (at 266.7 60.96) (diameter 0) (color 0 0 0 0)
   )
-  (junction (at 162.56 270.51) (diameter 0) (color 0 0 0 0)
-  )
   (junction (at 118.11 60.96) (diameter 0) (color 0 0 0 0)
   )
@@
     (stroke (width 0) (type default))
   )
+  (wire (pts (xy 198.12 267.97) (xy 210.82 267.97))
+    (stroke (width 0) (type default))
+  )
   (wire (pts (xy 227.33 114.3) (xy 227.33 116.84))
     (stroke (width 0) (type default))
@@
     (stroke (width 0) (type default))
   )
+  (wire (pts (xy 213.36 262.89) (xy 210.82 262.89))
+    (stroke (width 0) (type default))
+  )
   (wire (pts (xy 369.57 146.05) (xy 369.57 138.43))
     (stroke (width 0) (type default))
@@
     (stroke (width 0) (type default))
   )
+  (wire (pts (xy 198.12 257.81) (xy 213.36 257.81))
+    (stroke (width 0) (type default))
+  )
   (wire (pts (xy 114.3 259.08) (xy 114.3 242.57))
     (stroke (width 0) (type default))
@@
     (stroke (width 0) (type default))
   )
+  (wire (pts (xy 198.12 260.35) (xy 213.36 260.35))
+    (stroke (width 0) (type default))
+  )
   (wire (pts (xy 388.62 114.3) (xy 388.62 118.11))
     (stroke (width 0) (type default))
@@
     (stroke (width 0) (type default))
   )
+  (wire (pts (xy 213.36 267.97) (xy 213.36 273.05))
+    (stroke (width 0) (type default))
+  )
   (wire (pts (xy 78.74 104.14) (xy 78.74 106.68))
     (stroke (width 0) (type default))
@@
     (stroke (width 0) (type default))
   )
+  (wire (pts (xy 212.09 270.51) (xy 198.12 270.51))
+    (stroke (width 0) (type default))
+  )
   (wire (pts (xy 227.33 35.56) (xy 227.33 38.1))
     (stroke (width 0) (type default))
@@
     (stroke (width 0) (type default))
   )
+  (wire (pts (xy 210.82 262.89) (xy 210.82 267.97))
+    (stroke (width 0) (type default))
+  )
   (wire (pts (xy 144.78 22.86) (xy 144.78 25.4))
     (stroke (width 0) (type default))
@@
     (stroke (width 0) (type default))
   )
+  (wire (pts (xy 212.09 265.43) (xy 212.09 270.51))
+    (stroke (width 0) (type default))
+  )
   (wire (pts (xy 243.84 58.42) (xy 243.84 60.96))
     (stroke (width 0) (type default))
@@
     (stroke (width 0) (type default))
   )
+  (wire (pts (xy 213.36 265.43) (xy 212.09 265.43))
+    (stroke (width 0) (type default))
+  )
   (wire (pts (xy 364.49 148.59) (xy 372.11 148.59))
     (stroke (width 0) (type default))
@@
     (stroke (width 0) (type default))
   )
-  (wire (pts (xy 162.56 270.51) (xy 167.64 270.51))
-    (stroke (width 0) (type default))
-  )
   (wire (pts (xy 62.23 137.16) (xy 62.23 139.7))
     (stroke (width 0) (type default))
@@
     (effects (font (size 1.27 1.27)) (justify left bottom))
   )
+  (label "USBUP+" (at 266.7 231.14 0) (fields_autoplaced)
+    (effects (font (size 1.27 1.27)) (justify left bottom))
+  )
+  (label "USB3-" (at 364.49 191.77 0) (fields_autoplaced)
+    (effects (font (size 1.27 1.27)) (justify left bottom))
+  )
+  (label "USB2+" (at 109.22 240.03 0) (fields_autoplaced)
+    (effects (font (size 1.27 1.27)) (justify left bottom))
+  )
+  (label "USB2-" (at 109.22 242.57 0) (fields_autoplaced)
+    (effects (font (size 1.27 1.27)) (justify left bottom))
+  )
+  (label "USB4-" (at 364.49 102.87 0) (fields_autoplaced)
+    (effects (font (size 1.27 1.27)) (justify left bottom))
+  )
+  (label "USB3+" (at 364.49 196.85 0) (fields_autoplaced)
+    (effects (font (size 1.27 1.27)) (justify left bottom))
+  )
+  (label "USBUP-" (at 266.7 228.6 0) (fields_autoplaced)
+    (effects (font (size 1.27 1.27)) (justify left bottom))
+  )
+  (label "USB4+" (at 364.49 107.95 0) (fields_autoplaced)
+    (effects (font (size 1.27 1.27)) (justify left bottom))
+  )
   (global_label "I2C1-SCL" (shape input) (at 113.03 199.39 0) (fields_autoplaced)
     (effects (font (size 1.27 1.27)) (justify left))
@@
     )
   )
+  (symbol (lib_id "Connector:Conn_01x05_Socket") (at 218.44 262.89 0) (unit 1)
+    (in_bom yes) (on_board yes) (dnp no)
+    (property "Reference" "J10" (at 214.63 254 0)
+      (effects (font (size 1.27 1.27)) (justify left))
+    )
+    (property "Value" "Conn_01x05_Socket GPIOs" (at 219.71 271.78 90)
+      (effects (font (size 1.27 1.27)) (justify left))
+    )
+    (property "Footprint" "Connector_PinHeader_2.54mm:PinHeader_1x05_P2.54mm_Vertical" (at 218.44 262.89 0)
+      (effects (font (size 1.27 1.27)) hide)
+    )
+    (property "Datasheet" "~" (at 218.44 262.89 0)
+      (effects (font (size 1.27 1.27)) hide)
+    )
+    (pin "1")
+    (pin "2")
+    (pin "3")
+    (pin "4")
+    (pin "5")
+    (instances
+      (project "Quanta_RP2040Stamp_JLCPCBAoptimized"
+        (path "/0cabb2e6-4a46-4ffe-8ff7-d51fc1f6dda5"
+          (reference "J10") (unit 1)
+        )
+      )
+    )
+  )
   (symbol (lib_id "Device:R_Small") (at 370.84 92.71 90) (unit 1)
     (in_bom yes) (on_board yes) (dnp no)
@@
     )
   )
+  (symbol (lib_id "power:GND") (at 213.36 273.05 0) (unit 1)
+    (in_bom yes) (on_board yes) (dnp no)
+    (property "Reference" "#PWR031" (at 213.36 279.4 0)
+      (effects (font (size 1.27 1.27)) hide)
+    )
+    (property "Value" "GND" (at 213.36 276.86 0)
+      (effects (font (size 1.27 1.27)))
+    )
+    (property "Footprint" "" (at 213.36 273.05 0)
+      (effects (font (size 1.27 1.27)) hide)
+    )
+    (property "Datasheet" "" (at 213.36 273.05 0)
+      (effects (font (size 1.27 1.27)) hide)
+    )
+    (pin "1")
+    (instances
+      (project "Quanta_RP2040Stamp_JLCPCBAoptimized"
+        (path "/0cabb2e6-4a46-4ffe-8ff7-d51fc1f6dda5"
+          (reference "#PWR031") (unit 1)
+        )
+      )
+    )
+  )
   (symbol (lib_id "pspice:DIODE") (at 57.15 106.68 0) (mirror x) (unit 1)
     (in_bom yes) (on_board yes) (dnp no)
@@
     )
   )
-  (symbol (lib_id "Connector:Conn_01x01_Socket") (at 162.56 265.43 90) (unit 1)
-    (in_bom yes) (on_board yes) (dnp no)
-    (property "Reference" "J11" (at 163.83 265.43 90)
-      (effects (font (size 1.27 1.27)) (justify right))
-    )
-    (property "Value" "Conn_01x01_Socket GND" (at 148.59 262.89 90)
-      (effects (font (size 1.27 1.27)) (justify right))
-    )
-    (property "Footprint" "Connector_PinHeader_2.54mm:PinHeader_1x01_P2.54mm_Vertical" (at 162.56 265.43 0)
-      (effects (font (size 1.27 1.27)) hide)
-    )
-    (property "Datasheet" "~" (at 162.56 265.43 0)
-      (effects (font (size 1.27 1.27)) hide)
-    )
-    (pin "1")
-    (instances
-      (project "Quanta_RP2040Stamp_JLCPCBAoptimized"
-        (path "/0cabb2e6-4a46-4ffe-8ff7-d51fc1f6dda5"
-          (reference "J11") (unit 1)
-        )
-      )
-    )
-  )
   (symbol (lib_name "SW_Push_1") (lib_id "Switch:SW_Push") (at 210.82 99.06 90) (unit 1)
     (in_bom yes) (on_board yes) (dnp no)
@@
     )
   )
-  (symbol (lib_id "Connector:TestPoint") (at 162.56 270.51 180) (unit 1)
+  (symbol (lib_id "Connector:TestPoint") (at 167.64 270.51 0) (unit 1)
     (in_bom yes) (on_board yes) (dnp no)
-    (property "Reference" "TP5" (at 160.6272 275.6227 0)
+    (property "Reference" "TP5" (at 169.5728 265.3973 0)
       (effects (font (size 1.27 1.27)) (justify right))
     )
-    (property "Value" "GND" (at 160.4295 277.2439 0)
+    (property "Value" "GND" (at 169.7705 263.7761 0)
       (effects (font (size 1.27 1.27)) (justify right))
     )
-    (property "Footprint" "TestPoint:TestPoint_Pad_D1.5mm" (at 157.48 270.51 0)
+    (property "Footprint" "TestPoint:TestPoint_Pad_D1.5mm" (at 172.72 270.51 0)
       (effects (font (size 1.27 1.27)) hide)
     )
-    (property "Datasheet" "~" (at 157.48 270.51 0)
+    (property "Datasheet" "~" (at 172.72 270.51 0)
       (effects (font (size 1.27 1.27)) hide)
     )

Commit message: fine tune optimized pcb
Parts:
- removed J13: Conn_01x01_Socket GPIO0, Connector_PinHeader_2.54mm:PinHeader_1x01_P2.54mm_Vertical, symbol Connector:Conn_01x01_Socket
- added D87: Amber LED, LED_THT:LED_D5.0mm_Clear, symbol Device:LED
- added D88: Amber LED, LED_THT:LED_D3.0mm_Clear, symbol Device:LED
- added R12, R13, R15: 120R, Resistor_SMD:R_0603_1608Metric_Pad0.98x0.95mm_HandSolder, symbol Device:R
Connections:
- net GND: now also R15.2
- net GPIO0_LED: now reaches U1.1 (GPIO0)
- net GPIO0_LED: now also D87.2 (A), D88.2 (A)
- new net: R12.2, R13.1
- new net: R13.2, R15.1
- new net: D87.1 (K), D88.1 (K), R12.1
