File: Quanta_RP2040Stamp_JLCPCBAoptimized/Quanta_RP2040Stamp_JLCPCBAoptimized.kicad_pcb (KiCad board)
At the start: 2 copper layers, 317.5 x 163.5 mm, 226 parts, among them J1 USB_C_Receptacle_USB2.0, J10 USB_A_Receptacle_UBS2.0, J11 Conn_01x01_Socket GND, J12 Conn_01x06_Socket GPIOs, J13 Conn_01x01_Socket GPIO0, J2 Conn_01x02_Socket VBUS 5V, J3 Conn_01x02_Socket 3V3, J4 Conn_01x02_Socket VBAT, J5 Conn_01x04_Socket SWL, J6 USB_A_Receptacle_UBS2.0, J9 USB_C_Receptacle_USB2.0, SW1 SW_Push, SW10 SW_Push, SW11 SW_Push, SW12 SW_Push, SW13 SW_Push, SW14 SW_Push, SW15 SW_Push, SW16 SW_Push, SW17 SW_Push, SW18 SW_Push, SW19 SW_Push, SW2 SW_Push, SW20 SW_Push, SW21 SW_Push, SW22 SW_Push, SW23 SW_Push, SW24 SW_Push, SW25 SW_Push, SW26 SW_Push, SW27 SW_Push, SW28 SW_Push, SW29 SW_Push, SW3 SW_Push, SW30 SW_Push, SW31 SW_Push, SW32 SW_Push, SW33 SW_Push, SW34 SW_Push, SW35 SW_Push, SW36 SW_Push, SW37 SW_Push, SW38 SW_Push, SW39 SW_Push, SW4 SW_Push, SW40 SW_Push, SW41 SW_Push, SW42 SW_Push, SW43 SW_Push, SW44 SW_Push, SW45 SW_Push, SW46 SW_Push, SW47 SW_Push, SW48 SW_Push, SW49 SW_Push, SW5 SW_Push, SW50 SW_Push, SW51 SW_Push, SW52 SW_Push, SW53 SW_Push, SW54 SW_Push, SW55 SW_Push, SW56 SW_Push, SW57 SW_Push, SW58 SW_Push, SW59 SW_Push, SW6 SW_Push, SW60 SW_Push, SW61 SW_Push, SW62 SW_Push, SW63 SW_Push, SW64 SW_Push, SW65 SW_Push, SW66 SW_Push, SW67 SW_Push, SW68 SW_Push, SW69 SW_Push, SW7 SW_Push, SW70 SW_Push, SW71 SW_Push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

Commit message: update rev of optimized pcb
Parts:
- removed F1: 2A, Fuse:Fuse_1206_3216Metric_Pad1.42x1.75mm_HandSolder
- removed F3, F4: 500mA, Fuse:Fuse_1206_3216Metric_Pad1.42x1.75mm_HandSolder
- removed J10: USB_A_Receptacle_UBS2.0, USB_A_horizontal_SMD_903-231A2031S10100:USB-A-SMD_903-231A2031S10100
- removed R12: 0R, Resistor_SMD:R_1206_3216Metric_Pad1.30x1.75mm_HandSolder
- removed R13: 1M, Resistor_SMD:R_0805_2012Metric_Pad1.20x1.40mm_HandSolder
- added FB9: 100R 800mA, PCM_Ferrite_SMD_Handsoldering_AKL:Ferrite_0805_2012Metric_Pad1.05x1.20mm_BigPads, B.Cu at (247.1, 56.7)
- added J7: USB_C_Receptacle_USB2.0, USB_C_socket_GT-USB-7010H:USB-C-SMD_G-SWITCH_GT-USB-7010EN, B.Cu at (259.6, 69.8)
- added J8: Conn_01x04_Socket I2C display, Connector_PinHeader_2.54mm:PinHeader_1x04_P2.54mm_Vertical, F.Cu at (68.3, 87.5)
- added R14: 15k, Resistor_SMD:R_0603_1608Metric_Pad0.98x0.95mm_HandSolder, B.Cu at (243.5, 44.9)
- added R2: 4k99, Resistor_SMD:R_0603_1608Metric_Pad0.98x0.95mm_HandSolder, B.Cu at (252.2, 42.4)
- added R6: 15k, Resistor_SMD:R_0603_1608Metric_Pad0.98x0.95mm_HandSolder, B.Cu at (247.9, 39.8)
- added R7: 43k, Resistor_SMD:R_0603_1608Metric_Pad0.98x0.95mm_HandSolder, B.Cu at (247.9, 42.4)
- C1, C2, C3, C4, C7: footprint Capacitor_SMD:C_0805_2012Metric_Pad1.18x1.45mm_HandSolder -> Capacitor_SMD:C_0603_1608Metric_Pad1.08x0.95mm_HandSolder
- FB4: value 100R 2A5 -> 100R 800mA; footprint PCM_Ferrite_SMD_Handsoldering_AKL:Ferrite_0603_1608Metric -> PCM_Ferrite_SMD_Handsoldering_AKL:Ferrite_0805_2012Metric_Pad1.05x1.20mm_BigPads
- FB7: value 600R -> 600R 500mA
- FB8: value 600R 500mA -> 600R
- J5: value Conn_01x04_Socket SWL -> Conn_01x04_Socket SWD
- R1: value 0R -> 120R; footprint Resistor_SMD:R_1206_3216Metric_Pad1.30x1.75mm_HandSolder -> Resistor_SMD:R_0603_1608Metric_Pad0.98x0.95mm_HandSolder
- R10: value 56K 20% -> 43k
- R11: value 56K 20% -> 15k
- R3: value 5K11 -> 120R
- R4: value 5K11 -> 4k99
- R5: value 1M -> 43k; footprint Resistor_SMD:R_0805_2012Metric_Pad1.20x1.40mm_HandSolder -> Resistor_SMD:R_0603_1608Metric_Pad0.98x0.95mm_HandSolder
- R8: value 0R -> 43k; footprint Resistor_SMD:R_1206_3216Metric_Pad1.30x1.75mm_HandSolder -> Resistor_SMD:R_0603_1608Metric_Pad0.98x0.95mm_HandSolder
- R9: value 1M -> 15k; footprint Resistor_SMD:R_0805_2012Metric_Pad1.20x1.40mm_HandSolder -> Resistor_SMD:R_0603_1608Metric_Pad0.98x0.95mm_HandSolder
- RESW1: footprint Rotary_Encoder:RotaryEncoder_Bourns_Vertical_PEC12R-3xxxF-Sxxxx -> PEC12R-4120F-S0012:SW-TH_PEC12R-4120F-S0012
- moved R9 115.9 mm to (243.5, 37.3), turned to 180 degrees
- moved R11 106.8 mm to (243.5, 42.4), turned to 180 degrees
- moved R8 105.8 mm to (247.9, 44.9), turned to 180 degrees
- moved R10 104.5 mm to (243.5, 39.8), turned to 180 degrees
- moved FB7 103.2 mm to (236.7, 47.7), turned to 180 degrees
- moved FB8 101.3 mm to (236.7, 50.8), turned to 180 degrees
- moved C6 91.9 mm to (238.4, 37.8), turned to 180 degrees
- moved C2 85.8 mm to (252.2, 37.3), turned to 180 degrees
- moved R5 70.5 mm to (247.9, 37.3), turned to 180 degrees
- moved FB3 69.6 mm to (290.2, 38.2), turned to 180 degrees
- moved R1 66.4 mm to (252.2, 39.8)
- moved FB6 65.3 mm to (290.2, 41.3), turned to 180 degrees
- moved D86 64.5 mm to (260.4, 80.2)
- moved R3 60.1 mm to (252.2, 44.9), turned to 180 degrees
- moved C1 58.4 mm to (294.8, 34.8), turned to 180 degrees
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Connections:
- C6 pad 1: GND -> Net-(D86-VP)
- C6 pad 2: Net-(D86-VP) -> GND
- D86 pad 4: USB4_D- -> USB4_D+
- D86 pad 6: USB4_D+ -> USB4_D-
- FB1 pad 1: Net-(J1-SHIELD) -> GND
- FB1 pad 2: GND -> Net-(J1-SHIELD)
- FB2 pad 1: Net-(J6-Shield) -> GND
- FB2 pad 2: GND -> Net-(J6-Shield)
- FB3 pad 1: Net-(J9-SHIELD) -> GND
- FB3 pad 2: GND -> Net-(J9-SHIELD)
- FB4 pad 1: Net-(F1-Pad1) -> VBUS_UP
- FB5 pad 2: Net-(F2-Pad2) -> Net-(D84-VP)
- FB6 pad 2: Net-(F3-Pad2) -> Net-(D85-VP)
- FB7 pad 1: Net-(J10-Shield) -> +5V
- FB7 pad 2: GND -> Net-(D86-VP)
- FB8 pad 1: +5V -> GND
- R1 pad 1: GND -> Net-(R1-Pad1)
- R1 pad 2: Net-(J1-SHIELD) -> GND
- R10 pad 1: +5V -> Net-(J9-CC1)
- R10 pad 2: Net-(J9-CC1) -> Net-(R10-Pad2)
- R11 pad 1: +5V -> Net-(R11-Pad1)
- R11 pad 2: Net-(J9-CC2) -> +5V
- R3 pad 1: Net-(J1-CC2) -> Net-(R2-Pad2)
- R4 pad 2: GND -> Net-(R1-Pad1)
- R5 pad 1: GND -> Net-(J7-CC1)
- R5 pad 2: Net-(J1-SHIELD) -> Net-(R5-Pad2)
- R8 pad 1: GND -> Net-(J7-CC2)
- R8 pad 2: Net-(J9-SHIELD) -> Net-(R8-Pad2)
- R9 pad 1: GND -> Net-(R8-Pad2)
- R9 pad 2: Net-(J9-SHIELD) -> +5V
- U1 pad 25: Net-(J12-Pin_1) -> unconnected-(U1-GPIO24-Pad25)
- U1 pad 26: Net-(J12-Pin_2) -> unconnected-(U1-GPIO25-Pad26)
- U1 pad 27: Net-(J12-Pin_3) -> I2C1-SDA
- U1 pad 28: Net-(J12-Pin_4) -> I2C1-SCL
- U1 pad 29: Net-(J12-Pin_5) -> unconnected-(U1-GPIO28-Pad29)
- U1 pad 30: Net-(J12-Pin_6) -> unconnected-(U1-GPIO29-Pad30)
- U2 pad 1: USB4_D- -> USB2_D-
- U2 pad 2: USB4_D+ -> USB2_D+
- U2 pad 3: USB3_D- -> USB1_D-
- U2 pad 4: USB3_D+ -> USB1_D+
- U2 pad 5: USB2_D- -> USB4_D-
- U2 pad 6: USB2_D+ -> USB4_D+
- U2 pad 7: USB1_D- -> USB3_D-
- U2 pad 8: USB1_D+ -> USB3_D+
Routing:
- net +5V: track 93.2 -> 8.92 mm, vias 6 -> 0
- net VBUS_UP: track 41.3 -> 0.00 mm, vias 2 -> 0
- net Net-(D85-VP): track 37.9 -> 0.00 mm, vias 2 -> 0
- net Net-(D86-VP): track 21.4 -> 0.00 mm, vias 2 -> 0
- net Net-(D85-L1-Pad1): track 21.2 -> 0.00 mm
- net USB_UP_D+: track 19.9 -> 0.00 mm
- net USB_UP_D-: track 19.8 -> 0.00 mm
- net Net-(D86-L2-Pad3): track 19.7 -> 0.00 mm, vias 2 -> 0
- net Net-(D86-L1-Pad1): track 19.5 -> 0.00 mm, vias 2 -> 0
- net Net-(D85-L2-Pad3): track 18.7 -> 0.00 mm
- net Net-(U2-VDD18): track 10.5 -> 0.00 mm
- net Net-(J9-SHIELD): track 10.3 -> 0.00 mm
- net Net-(U2-VDD33): track 9.31 -> 0.00 mm
- net Net-(J1-SHIELD): track 8.03 -> 0.00 mm
- net Net-(J10-Shield): track 6.23 -> 0.00 mm
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Other:
- outline, holes or cut-outs redrawn
- board text removed: "UPSTREAM"

Commit message: routed matrix for optimized version
Parts:
- removed J11: Conn_01x01_Socket GND, Connector_PinHeader_2.54mm:PinHeader_1x01_P2.54mm_Vertical
- removed J12: Conn_01x06_Socket GPIOs, Connector_PinHeader_2.54mm:PinHeader_1x06_P2.54mm_Vertical
- removed the R2 at (337.3, 110.3)
- removed the R6 at (338.1, 114.6)
- added J10: Conn_01x05_Socket GPIOs, Connector_PinHeader_2.54mm:PinHeader_1x05_P2.54mm_Vertical, F.Cu at (167.5, 85.2)
- moved R3 95.6 mm to (342.0, 77.9), turned to -90 degrees
- moved R2 95.1 mm to (341.8, 74.2), turned to -90 degrees
- moved R1 94.9 mm to (339.2, 77.8), turned to -90 degrees
- moved C2 93.8 mm to (325.4, 96.0), turned to 0 degrees
- moved FB9 84.8 mm to (329.8, 75.6), turned to -90 degrees
- moved FB1 68.3 mm to (348.2, 71.1)
- moved C1 66.5 mm to (325.4, 93.8), turned to 0 degrees
- moved TP11 64.2 mm to (329.4, 95.2), turned to 90 degrees
- moved TP12 62.8 mm to (325.4, 99.3), turned to 0 degrees
- moved C3 62.1 mm to (325.5, 91.3), turned to 0 degrees
- moved R4 53.2 mm to (339.2, 74.2), turned to -90 degrees
- moved C4 51.7 mm to (334.1, 73.5), turned to -90 degrees
- moved C7 51.0 mm to (330.7, 78.6)
- moved FB4 47.8 mm to (332.1, 75.6), turned to -90 degrees
- moved C9 38.2 mm to (326.2, 80.2), turned to 90 degrees
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Connections:
- net Net-(D85-L1-Pad1) renamed /USB3-
- net Net-(D85-L2-Pad3) renamed /USB3+
- net Net-(D86-L1-Pad1) renamed /USB4-
- net Net-(D86-L2-Pad3) renamed /USB4+
- net Net-(J6-D+) renamed /USB2+
- net Net-(J6-D-) renamed /USB2-
- net Net-(U2-DM) renamed /USBUP-
- net Net-(U2-DP) renamed /USBUP+
- U1 pad 25: unconnected-(U1-GPIO24-Pad25) -> Net-(J10-Pin_1)
- U1 pad 26: unconnected-(U1-GPIO25-Pad26) -> Net-(J10-Pin_2)
- U1 pad 29: unconnected-(U1-GPIO28-Pad29) -> Net-(J10-Pin_3)
- U1 pad 30: unconnected-(U1-GPIO29-Pad30) -> Net-(J10-Pin_4)
Routing:
- net Row6: track 0.00 -> 308.5 mm
- net Row1: track 0.00 -> 304.7 mm
- net Row3: track 0.00 -> 301.9 mm
- net Row5: track 0.00 -> 301.3 mm
- net Row2: track 0.00 -> 299.8 mm
- net Row4: track 0.00 -> 292.7 mm
- net +3.3V: track 25.2 -> 187.7 mm, vias 0 -> 1
- net I2C1-SCL: track 0.00 -> 145.4 mm
- net I2C1-SDA: track 0.00 -> 137.9 mm
- net Column11: track 0.00 -> 137.0 mm
- net Column12: track 0.00 -> 136.6 mm
- net Column10: track 0.00 -> 136.3 mm
- net Column13: track 0.00 -> 132.1 mm
- net Column7: track 0.00 -> 123.6 mm
- net Column3: track 0.00 -> 121.9 mm
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Other:
- outline, holes or cut-outs redrawn
- board text added: "0bsilab"
- board text added: "Quanta"

Commit message: finished optimized pcb
Parts:
- moved TP4 87.8 mm to (220.7, 75.4), turned to -90 degrees
- moved R11 68.7 mm to (302.1, 78.4), turned to -90 degrees
- moved R10 65.5 mm to (299.2, 74.4), turned to -90 degrees
- moved R14 64.7 mm to (299.1, 77.9), turned to -90 degrees
- moved R7 63.3 mm to (302.1, 75.0), turned to -90 degrees
- moved TP14 54.2 mm to (346.7, 74.8)
- moved R9 45.5 mm to (261.6, 79.0), turned to -90 degrees
- moved C6 40.7 mm to (253.9, 75.3)
- moved R6 40.5 mm to (258.5, 78.9), turned to -90 degrees
- moved TP13 39.6 mm to (329.7, 70.6)
- moved R5 39.5 mm to (258.5, 75.4), turned to -90 degrees
- moved FB6 35.9 mm to (295.0, 76.9), turned to 0 degrees
- moved FB7 34.9 mm to (254.4, 77.7), turned to 0 degrees
- moved R8 33.6 mm to (261.6, 75.5), turned to -90 degrees
- moved C5 18.3 mm to (294.5, 74.6)
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Connections:
- J9 pad 2: (no net) -> Net-(J9-SHIELD)
Routing:
- net Row6: track 308.5 -> 574.9 mm
- net Row5: track 301.3 -> 545.1 mm
- net REB: track 0.00 -> 220.6 mm, vias 0 -> 3
- net REA: track 0.00 -> 220.2 mm, vias 0 -> 3
- net Row4: track 292.7 -> 511.9 mm
- net Row3: track 301.9 -> 496.7 mm
- net Column15: track 100.3 -> 283.0 mm
- net +5V: track 32.2 -> 210.0 mm, vias 2 -> 10
- net Row2: track 299.8 -> 470.2 mm, vias 0 -> 2
- net Column14: track 86.9 -> 242.3 mm
- net Row1: track 304.7 -> 446.3 mm
- net Column1: track 104.9 -> 240.4 mm
- net Column13: track 132.1 -> 258.8 mm
- net USB1_D+: track 0.00 -> 117.4 mm, vias 0 -> 2
- net USB1_D-: track 0.00 -> 117.4 mm, vias 0 -> 2
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Other:
- board size 317.5 x 163.5 mm -> 320.7 x 163.5 mm
- board text added: "ISO ENTER"
- board text added: "by Lucas Placentino"
- board text added: "https://github.com/ObsiLab/Quanta"
- board text added: "https://quanta.obsilab.com/"

Commit message: fine tune optimized pcb
Parts:
- removed J13: Conn_01x01_Socket GPIO0, Connector_PinHeader_2.54mm:PinHeader_1x01_P2.54mm_Vertical
- added D87: Amber LED, LED_THT:LED_D5.0mm_Clear, F.Cu at (337.2, 146.6)
- added D88: Amber LED, LED_THT:LED_D3.0mm_Clear, F.Cu at (337.2, 141.1)
- added M2.5: MountingHole_2.7mm_M2.5_DIN965_Pad, MountingHole:MountingHole_2.7mm_M2.5_DIN965_Pad, F.Cu at (50.0, 69.8)
- added M2.5: MountingHole_2.7mm_M2.5_DIN965_Pad, MountingHole:MountingHole_2.7mm_M2.5_DIN965_Pad, F.Cu at (210.3, 214.3)
- added M2.5: MountingHole_2.7mm_M2.5_DIN965_Pad, MountingHole:MountingHole_2.7mm_M2.5_DIN965_Pad, F.Cu at (338.1, 153.2)
- added M2.5: MountingHole_2.7mm_M2.5_DIN965_Pad, MountingHole:MountingHole_2.7mm_M2.5_DIN965_Pad, F.Cu at (138.9, 124.6)
- added M2.5: MountingHole_2.7mm_M2.5_DIN965_Pad, MountingHole:MountingHole_2.7mm_M2.5_DIN965_Pad, F.Cu at (361.2, 225.4)
- added M2.5: MountingHole_2.7mm_M2.5_DIN965_Pad, MountingHole:MountingHole_2.7mm_M2.5_DIN965_Pad, F.Cu at (77.0, 177.0)
- added M2.5: MountingHole_2.7mm_M2.5_DIN965_Pad, MountingHole:MountingHole_2.7mm_M2.5_DIN965_Pad, F.Cu at (252.4, 124.3)
- added M2.5: MountingHole_2.7mm_M2.5_DIN965_Pad, MountingHole:MountingHole_2.7mm_M2.5_DIN965_Pad, F.Cu at (122.7, 212.7)
- added M2.5: MountingHole_2.7mm_M2.5_DIN965_Pad, MountingHole:MountingHole_2.7mm_M2.5_DIN965_Pad, F.Cu at (361.2, 69.8)
- added M2.5: MountingHole_2.7mm_M2.5_DIN965_Pad, MountingHole:MountingHole_2.7mm_M2.5_DIN965_Pad, F.Cu at (50.0, 225.4)
- added M6Hole: MountingHole_6.4mm_M6_DIN965, MountingHole:MountingHole_6.4mm_M6_DIN965, F.Cu at (231.8, 123.8)
- added M6Hole: MountingHole_6.4mm_M6_DIN965, MountingHole:MountingHole_6.4mm_M6_DIN965, F.Cu at (69.8, 123.8)
- added M6Hole: MountingHole_6.4mm_M6_DIN965, MountingHole:MountingHole_6.4mm_M6_DIN965, F.Cu at (56.4, 76.2)
- added M6Hole: MountingHole_6.4mm_M6_DIN965, MountingHole:MountingHole_6.4mm_M6_DIN965, F.Cu at (219.1, 211.9)
- added M6Hole: MountingHole_6.4mm_M6_DIN965, MountingHole:MountingHole_6.4mm_M6_DIN965, F.Cu at (338.9, 127.8)
- added M6Hole: MountingHole_6.4mm_M6_DIN965, MountingHole:MountingHole_6.4mm_M6_DIN965, F.Cu at (225.4, 92.9)
- added M6Hole: MountingHole_6.4mm_M6_DIN965, MountingHole:MountingHole_6.4mm_M6_DIN965, F.Cu at (72.2, 222.2)
- added M6Hole: MountingHole_6.4mm_M6_DIN965, MountingHole:MountingHole_6.4mm_M6_DIN965, F.Cu at (297.7, 223.0)
- added M6Hole: MountingHole_6.4mm_M6_DIN965, MountingHole:MountingHole_6.4mm_M6_DIN965, F.Cu at (354.8, 76.2)
- added OSHW-logo: OSHW-Logo_19x20mm_Copper, Symbol:OSHW-Logo_19x20mm_Copper, B.Cu at (134.9, 83.3)
- added Quanta***: LOGO, Quanta-logo:Quanta-logo, F.Cu at (192.7, 86.3)
- added R12: 120R, Resistor_SMD:R_0603_1608Metric_Pad0.98x0.95mm_HandSolder, B.Cu at (332.7, 144.5)
- added R13: 120R, Resistor_SMD:R_0603_1608Metric_Pad0.98x0.95mm_HandSolder, B.Cu at (332.6, 141.3)
- added R15: 120R, Resistor_SMD:R_0603_1608Metric_Pad0.98x0.95mm_HandSolder, B.Cu at (332.6, 138.1)
- added REF**: OSHW-Logo_19x20mm_Copper, Symbol:OSHW-Logo_19x20mm_Copper, F.Cu at (279.4, 82.5)
- moved J7 0.79 mm to (259.6, 69.1)
Connections:
- J7 pad 2: (no net) -> Net-(J7-SHIELD)
- J9 pad 2: Net-(J9-SHIELD) -> (no net)
- RESW1 pad 1: Net-(RED1-A) -> (no net)
- RESW1 pad 2: Row1 -> (no net)
- U1 pad 1: Net-(J13-Pin_1) -> GPIO0_LED
Routing:
- net (no net): track 0.00 -> 209.2 mm
- net GPIO0_LED: track 0.00 -> 169.4 mm, vias 0 -> 4
- net Net-(J7-SHIELD): track 2.80 -> 156.5 mm
- net Net-(D87-K): track 0.00 -> 10.1 mm
- net Net-(D86-VP): track 18.5 -> 28.6 mm, vias 0 -> 2
- net Net-(D85-VP): track 15.4 -> 24.1 mm, vias 0 -> 2
- net Net-(J13-Pin_1): track 8.23 -> 0.00 mm
- net Net-(R12-Pad2): track 0.00 -> 3.22 mm
- net Net-(R13-Pad2): track 0.00 -> 3.17 mm
- net /USB4-: track 15.1 -> 16.3 mm
- net /USB4+: track 16.1 -> 17.0 mm
- net Net-(J7-CC2): track 2.51 -> 3.30 mm
- net Net-(J7-CC1): track 2.30 -> 3.09 mm
Other:
- board size 320.7 x 163.5 mm -> 320.7 x 165.1 mm
- board text added: "3V3"
- board text added: "CAPS LOCK"
- board text added: "GND"
- board text added: "GPIO25"
- board text added: "GPIO26"
- board text added: "GPIO29"
- board text added: "GPIO30"
- board text added: "I²C OLED"
- board text added: "MX style switches and stabs only"
- board text added: "PEC12R-4-S"
- board text added: "ROTARY ENCODER"
- board text added: "SCL"
- board text added: "SDA"
- board text added: "UPSTREAM"
- board text added: "USB nb2"
- board text added: "USB nb3"
- board text added: "USB nb4"
- board text added: "Use Mill-Max 3305 hotswap to add hotswap fonctionality"
- board text added: "or"

Commit message: fix
Parts:
- moved OSHW-logo 144.5 mm to (279.4, 82.5)
Changed lines of the file:
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@@
   )
   (footprint "Symbol:OSHW-Logo_19x20mm_Copper" (layer "B.Cu")
-    (at 134.9375 83.34375 180)
+    (at 279.4 82.55 180)
     (descr "Open Source Hardware Logo")
     (tags "Logo OSHW")
